Commit message: created a new base urdf to plan

File: robotino_description/urdf/base_plan.urdf.xacro (robot description, xacro)
@@ -3,18 +3,67 @@
   <xacro:include filename="$(find robotino_description)/urdf/gazebo.urdf.xacro" />
   <xacro:macro name="base" params="name">
-    <!--link name="${name}_footprint">
-   <visual>
+   <link name="${name}_link">
+      <inertial>
+        <mass value="10" />
+        <origin xyz="0 0 0" />
+        <inertia ixx="75.0" ixy="0.0" ixz="0.0"
+          iyy="75.0" iyz="0.0"
+          izz="75.0" />
+      </inertial>
+    </link>
+    <joint name="${name}_jointx" type="prismatic">
+      <parent link="${name}_link"/>
+      <child link="${name}_linkx"/>
       <origin xyz="0 0 0" rpy="0 0 0" />
-      <geometry>
-        <box size="0.001 0.001 0.001" />
-      </geometry>
-    </visual>
-  </link>
-   <joint name="${name}_footprint_joint" type="fixed">
+      <axis xyz="1 0 0" />
+      <limit upper="10" lower="-10" effort="190" velocity="30" />
+    </joint>
+   <link name="${name}_linkx">
+      <inertial>
+        <mass value="10" />
+        <origin xyz="0 0 0" />
+        <inertia ixx="75.0" ixy="0.0" ixz="0.0"
+          iyy="75.0" iyz="0.0"
+          izz="75.0" />
+      </inertial>
+    </link>
+    <joint name="${name}_jointy" type="prismatic">
+      <parent link="${name}_linkx"/>
+      <child link="${name}_linky"/>
       <origin xyz="0 0 0" rpy="0 0 0" />
-      <child link="${name}_link" />
-      <parent link="${name}_footprint"/>
-   </joint-->
-   <link name="${name}_link">
+      <axis xyz="0 1 0" />
+      <limit upper="10" lower="-10" effort="190" velocity="30" />
+    </joint>
+   <link name="${name}_linky">
+      <inertial>
+        <mass value="10" />
+        <origin xyz="0 0 0" />
+        <inertia ixx="75.0" ixy="0.0" ixz="0.0"
+          iyy="75.0" iyz="0.0"
+          izz="75.0" />
+      </inertial>
+    </link>
+    <joint name="${name}_jointz" type="revolute">
+      <parent link="${name}_linky"/>
+      <child link="${name}_linkz"/>
+      <origin xyz="0 0 0" rpy="0 0 0" />
+      <axis xyz="0 0 1" />
+      <limit upper="3.14" lower="-3.14" effort="190" velocity="30" />
+    </joint>
+   <link name="${name}_linkz">
+      <inertial>
+        <mass value="10" />
+        <origin xyz="0 0 0" />
+        <inertia ixx="75.0" ixy="0.0" ixz="0.0"
+          iyy="75.0" iyz="0.0"
+          izz="75.0" />
+      </inertial>
+    </link>
+    <joint name="${name}_body_joint" type="fixed">
+      <parent link="${name}_linkz"/>
+      <child link="${name}_body_link"/>
+      <origin xyz="0 0 0" rpy="0 0 0" />
+    </joint>
+   <link name="${name}_body_link">
       <inertial>
         <mass value="10" />
@@ -38,5 +87,5 @@
     </link>
     <base_gazebo name="base" />
-    <wheel name="wheel0" parent="base_link">
+    <wheel name="wheel0" parent="base_linkz">
       <origin xyz="0.095 0.14 0.02" rpy="0 0 ${M_PI/3}"/>
       <axis xyz="-1 0 0"/>
@@ -44,5 +93,5 @@
     <wheel_transmission name="wheel0" />
     <wheel_gazebo name="wheel0" />
-    <wheel name="wheel1" parent="base_link">
+    <wheel name="wheel1" parent="base_linkz">
       <origin xyz="-0.16 0 0.02" rpy="0 0 0"/>
       <axis xyz="1 0 0"/>
@@ -50,5 +99,5 @@
     <wheel_transmission name="wheel1" />
     <wheel_gazebo name="wheel1" />
-    <wheel name="wheel2" parent="base_link">
+    <wheel name="wheel2" parent="base_linkz">
       <origin xyz="0.105 -0.15 0.02" rpy="0 0 -${M_PI/3}"/>
       <axis xyz="-1 0 0"/>
@@ -100,3 +149,15 @@
     </transmission>
   </xacro:macro>
+  <xacro:macro name="joints_transmission" params="name">
+    <transmission name="${name}_trans">
+      <type>transmission_interface/SimpleTransmission</type>
+      <joint name="${name}" >
+        <hardwareInterface>VelocityJointInterface</hardwareInterface>
+      </joint>
+      <actuator name="${name}_motor">
+        <hardwareInterface>VelocityJointInterface</hardwareInterface>
+        <mechanicalReduction>${ 624/35 * 80/18}</mechanicalReduction>
+      </actuator>
+    </transmission>
+  </xacro:macro>
 </root>

Commit message: simplify collision model

File: robotino_description/urdf/base_plan.urdf.xacro (robot description, xacro)
@@ -80,7 +80,7 @@
       </visual>
       <collision>
-        <origin xyz="0.01 0 0" rpy="0 0 0"/>
+        <origin xyz="0.01 0 0.12" rpy="0 0 0"/>
         <geometry>
-          <mesh filename="package://robotino_description/meshes/RobotinoBody.stl"/>
+          <cylinder length="0.24" radius="0.23"/>
         </geometry>
       </collision>
