Commit message: colored the shell

File: robotino_description/urdf/base_shell.urdf.xacro (robot description, xacro)
@@ -20,4 +20,7 @@
           <mesh filename="package://robotino_description/meshes/squirrel_assembly.stl"/>
         </geometry>
+        <material name="lightGrey">
+          <color rgba="0.9 0.9 0.9 1"/>
+        </material>
       </visual>
       <collision>
@@ -28,4 +31,9 @@
       </collision>
     </link>
+    <gazebo reference="${name}_link">
+      <gravity>true</gravity>
+      <self_collide>false</self_collide>
+      <material>Gazebo/LightGrey</material>
+    </gazebo>
   </xacro:macro>
 </root>

Commit message: Temporal fix: ignore the visual model of the shell

File: robotino_description/urdf/base_shell.urdf.xacro (robot description, xacro)
@@ -15,5 +15,5 @@
           izz="75.0" />
       </inertial>
-      <visual>
+      <!--visual>
         <origin xyz="0 0 -0.04" rpy="0 0 0"/>
         <geometry>
@@ -23,5 +23,5 @@
           <color rgba="0.9 0.9 0.9 1"/>
         </material>
-      </visual>
+      </visual-->
       <collision>
         <origin xyz="0 0 0.05" rpy="0 0 -0.7"/>

Commit message: use rosindustrial ci config

File: robotino_description/urdf/base_shell.urdf.xacro (robot description, xacro)
@@ -15,5 +15,5 @@
           izz="75.0" />
       </inertial>
-      <!--visual>
+      <visual>
         <origin xyz="0 0 -0.04" rpy="0 0 0"/>
         <geometry>
@@ -23,5 +23,5 @@
           <color rgba="0.9 0.9 0.9 1"/>
         </material>
-      </visual-->
+      </visual>
       <collision>
         <origin xyz="0 0 0.05" rpy="0 0 -0.7"/>
