Commit message: reference frame for kclhand

File: robotino_description/urdf/kclhand_withCableCanal.urdf.xacro (robot description, xacro)
@@ -26,9 +26,15 @@
   </link>
   <joint name="${name}_base_joint" type="fixed">
+    <origin xyz="-0.02105 0.1485 0" rpy="-1.5708 0 0"/>
+    <parent link="${name}_wrist_link"/>
+    <child link="${name}_base_link"/>
+  </joint>
+  <link name="${name}_base_link"/>
+  <joint name="kcl${name}_base_joint" type="fixed">
     <origin xyz="-0.02105 0.1485 0" rpy="0 0.52 0"/>
     <parent link="${name}_wrist_link"/>
-    <child link="${name}_base_link"/>
-  </joint>
-  <link name="${name}_base_link">
+    <child link="kcl${name}_base_link"/>
+  </joint>
+  <link name="kcl${name}_base_link">
     <xacro:default_inertial/>
     <visual>
@@ -50,5 +56,5 @@
   <joint name="${name}_middle_finger_lower_joint" type="continuous">
     <origin xyz="0.035507 0.02 0.0205" rpy="-0.5236 5.5511E-17 1.5708"/>
-    <parent link="${name}_base_link"/>
+    <parent link="kcl${name}_base_link"/>
     <child link="${name}_middle_finger_lower_link"/>
     <axis xyz="0 0 -1"/>
@@ -98,5 +104,5 @@
   <joint name="${name}_left_crank_base_joint" type="continuous">
     <origin xyz="0 0 0" rpy="-2.1588 0.44783 -1.8518"/>
-    <parent link="${name}_base_link"/>
+    <parent link="kcl${name}_base_link"/>
     <child link="${name}_left_crank"/>
     <axis xyz="0 0 1"/>
@@ -194,5 +200,5 @@
   <joint name="${name}_right_crank_base_joint" type="continuous">
     <origin xyz="0 0 0" rpy="-5.5511E-17 -2.7756E-17 1.0472"/>
-    <parent link="${name}_base_link"/>
+    <parent link="kcl${name}_base_link"/>
     <child link="${name}_right_crank"/>
     <axis xyz="0 0 1"/>
@@ -321,5 +327,5 @@
   <xacro:kclhand_transmission name="${name}_right_finger_lower"/>
   <xacro:kclhand_transmission name="${name}_right_finger_upper"/>
-  <xacro:kclhand_gazebo name="${name}_base_link"/>
+  <xacro:kclhand_gazebo name="kcl${name}_base_link"/>
   <xacro:kclhand_gazebo name="${name}_left_coupler"/>
   <xacro:kclhand_gazebo name="${name}_left_crank"/>

Commit message: added hand_palm_link

File: robotino_description/urdf/kclhand_withCableCanal.urdf.xacro (robot description, xacro)
@@ -25,16 +25,16 @@
     </collision>
   </link>
+  <joint name="${name}_palm_joint" type="fixed">
+    <origin xyz="-0.02105 0.0485 0" rpy="-1.5708 0 0"/>
+    <parent link="${name}_wrist_link"/>
+    <child link="${name}_palm_link"/>
+  </joint>
+  <link name="${name}_palm_link"/>
   <joint name="${name}_base_joint" type="fixed">
-    <origin xyz="-0.02105 0.1485 0" rpy="-1.5708 0 0"/>
+    <origin xyz="-0.02105 0.1485 0" rpy="0 0.52 0"/>
     <parent link="${name}_wrist_link"/>
     <child link="${name}_base_link"/>
   </joint>
-  <link name="${name}_base_link"/>
-  <joint name="kcl${name}_base_joint" type="fixed">
-    <origin xyz="-0.02105 0.1485 0" rpy="0 0.52 0"/>
-    <parent link="${name}_wrist_link"/>
-    <child link="kcl${name}_base_link"/>
-  </joint>
-  <link name="kcl${name}_base_link">
+  <link name="${name}_base_link">
     <xacro:default_inertial/>
     <visual>
@@ -56,5 +56,5 @@
   <joint name="${name}_middle_finger_lower_joint" type="continuous">
     <origin xyz="0.035507 0.02 0.0205" rpy="-0.5236 5.5511E-17 1.5708"/>
-    <parent link="kcl${name}_base_link"/>
+    <parent link="${name}_base_link"/>
     <child link="${name}_middle_finger_lower_link"/>
     <axis xyz="0 0 -1"/>
@@ -104,5 +104,5 @@
   <joint name="${name}_left_crank_base_joint" type="continuous">
     <origin xyz="0 0 0" rpy="-2.1588 0.44783 -1.8518"/>
-    <parent link="kcl${name}_base_link"/>
+    <parent link="${name}_base_link"/>
     <child link="${name}_left_crank"/>
     <axis xyz="0 0 1"/>
@@ -200,5 +200,5 @@
   <joint name="${name}_right_crank_base_joint" type="continuous">
     <origin xyz="0 0 0" rpy="-5.5511E-17 -2.7756E-17 1.0472"/>
-    <parent link="kcl${name}_base_link"/>
+    <parent link="${name}_base_link"/>
     <child link="${name}_right_crank"/>
     <axis xyz="0 0 1"/>
@@ -327,5 +327,5 @@
   <xacro:kclhand_transmission name="${name}_right_finger_lower"/>
   <xacro:kclhand_transmission name="${name}_right_finger_upper"/>
-  <xacro:kclhand_gazebo name="kcl${name}_base_link"/>
+  <xacro:kclhand_gazebo name="${name}_base_link"/>
   <xacro:kclhand_gazebo name="${name}_left_coupler"/>
   <xacro:kclhand_gazebo name="${name}_left_crank"/>

Commit message: Update kclhand_withCableCanal.urdf.xacro

File: robotino_description/urdf/kclhand_withCableCanal.urdf.xacro (robot description, xacro)
@@ -26,5 +26,5 @@
   </link>
   <joint name="${name}_palm_joint" type="fixed">
-    <origin xyz="-0.02105 0.0485 0" rpy="-1.5708 0 0"/>
+    <origin xyz="-0.02105 0.2485 0" rpy="-1.5708 0 0"/> <!--palm_link.y(0.2485) = base_link.y(0.1485) + 0.1m-->
     <parent link="${name}_wrist_link"/>
     <child link="${name}_palm_link"/>
