Commit message: use a simple base for non-arm robots

File: robotino_description/urdf/base.gazebo.xacro (robot description, xacro)
@@ -38,5 +38,5 @@
       <gravity>true</gravity>
       <self_collide>false</self_collide>
-      <!--sensor name='${name}_contact_sensor' type='contact'>
+      <sensor name='${name}_contact_sensor' type='contact'>
         <always_on>true</always_on>
         <update_rate>1</update_rate>
@@ -49,5 +49,5 @@
           <bumperTopicName>${name}_bumper</bumperTopicName>
         </plugin>
-      </sensor-->
+      </sensor>
     </gazebo>
     <gazebo reference="${name}_link">
@@ -56,13 +56,4 @@
       <self_collide>false</self_collide>
     </gazebo>
-  <gazebo>
-    <plugin name="base_controller" filename="libgazebo_ros_planar_move.so">
-      <commandTopic>cmd_vel</commandTopic>
-      <odometryTopic>odom</odometryTopic>
-      <odometryFrame>odom</odometryFrame>
-      <odometryRate>20.0</odometryRate>
-      <robotBaseFrame>base_linkz</robotBaseFrame>
-    </plugin>
-  </gazebo>
   </xacro:macro>
 </robot>

File: robotino_description/urdf/base.urdf.xacro (robot description, xacro)
@@ -4,4 +4,6 @@
   <xacro:include filename="$(find robotino_description)/urdf/base.transmission.xacro" />
   <xacro:macro name="base" params="name has_8dof">
+  <!--###### IF 8 DOF the joints can be moved ######-->
+  <xacro:if value="${has_8dof}">
   <link name="origin" />
   <joint name="origin_joint" type="fixed">
@@ -19,6 +21,4 @@
     </inertial>
    </link>
-  <!--###### IF 8 DOF the joints can be moved ######-->
-  <xacro:if value="${has_8dof}">
    <joint name="${name}_jointx" type="prismatic">
     <parent link="origin"/>
@@ -51,23 +51,4 @@
    </joint>
    <joints_transmission name="base_jointz" />
-  </xacro:if>
-  <!--###### ELSE the joints are fixed ######-->
-  <xacro:unless value="${has_8dof}">
-   <joint name="${name}_jointx" type="fixed">
-    <parent link="origin"/>
-    <child link="${name}_linkx"/>
-    <origin xyz="0 0 0" rpy="0 0 0" />
-   </joint>
-   <joint name="${name}_jointy" type="fixed">
-    <parent link="${name}_linkx"/>
-    <child link="${name}_linky"/>
-    <origin xyz="0 0 0" rpy="0 0 0" />
-   </joint>
-   <joint name="${name}_jointz" type="fixed">
-    <parent link="${name}_linky"/>
-    <child link="${name}_linkz"/>
-    <origin xyz="0 0 0" rpy="0 0 0" />
-   </joint>
-  </xacro:unless>
   <link name="${name}_linkx">
    <inertial>
@@ -154,4 +135,13 @@
    </link>
    <base_gazebo name="base" />
+  <gazebo>
+    <plugin name="base_controller" filename="libgazebo_ros_planar_move.so">
+      <commandTopic>cmd_vel</commandTopic>
+      <odometryTopic>odom</odometryTopic>
+      <odometryFrame>odom</odometryFrame>
+      <odometryRate>20.0</odometryRate>
+      <robotBaseFrame>base_linkz</robotBaseFrame>
+    </plugin>
+  </gazebo>
    <wheel name="wheel0" parent="base_linkz">
     <origin xyz="0.095 0.14 0.02" rpy="0 0 ${M_PI/3}"/>
@@ -172,4 +162,63 @@
    <wheel_transmission name="wheel2" />
    <wheel_gazebo name="wheel2" />
+  </xacro:if>
+ <!--###### ELSE the joints are fixed ######-->
+  <xacro:unless value="${has_8dof}">
+  <link name="${name}_link" />
+   <joint name="${name}_body_joint" type="fixed">
+    <parent link="${name}_link"/>
+    <child link="${name}_body_link"/>
+    <origin xyz="0 0 0" rpy="0 0 0" />
+   </joint>
+  <link name="${name}_body_link">
+    <inertial>
+      <mass value="10" />
+      <origin xyz="0 0 0" />
+      <inertia ixx="75.0" ixy="0.0" ixz="0.0"
+       iyy="75.0" iyz="0.0"
+       izz="75.0" />
+    </inertial>
+    <visual>
+      <origin xyz="0.01 0 0" rpy="0 0 0"/>
+      <geometry>
+       <mesh filename="package://robotino_description/meshes/RobotinoBody.dae"/>
+      </geometry>
+    </visual>
+    <collision>
+      <origin xyz="0.01 0 0" rpy="0 0 0"/>
+      <geometry>
+       <mesh filename="package://robotino_description/meshes/RobotinoBody.stl"/>
+      </geometry>
+    </collision>
+   </link>
+   <base_gazebo name="base" />
+  <gazebo>
+    <plugin name="base_controller" filename="libgazebo_ros_planar_move.so">
+      <commandTopic>cmd_vel</commandTopic>
+      <odometryTopic>odom</odometryTopic>
+      <odometryFrame>odom</odometryFrame>
+      <odometryRate>20.0</odometryRate>
+      <robotBaseFrame>base_link</robotBaseFrame>
+    </plugin>
+  </gazebo>
+   <wheel name="wheel0" parent="base_link">
+    <origin xyz="0.095 0.14 0.02" rpy="0 0 ${M_PI/3}"/>
+    <axis xyz="-1 0 0"/>
+   </wheel>
+   <wheel_transmission name="wheel0" />
+   <wheel_gazebo name="wheel0" />
+   <wheel name="wheel1" parent="base_link">
+    <origin xyz="-0.16 0 0.02" rpy="0 0 0"/>
+    <axis xyz="1 0 0"/>
+   </wheel>
+   <wheel_transmission name="wheel1" />
+   <wheel_gazebo name="wheel1" />
+   <wheel name="wheel2" parent="base_link">
+    <origin xyz="0.105 -0.15 0.02" rpy="0 0 -${M_PI/3}"/>
+    <axis xyz="-1 0 0"/>
+   </wheel>
+   <wheel_transmission name="wheel2" />
+   <wheel_gazebo name="wheel2" />
+  </xacro:unless>
   </xacro:macro>
   <!-- WHEEL -->

Commit message: clean base URDF model

File: robotino_description/urdf/base.gazebo.xacro (robot description, xacro)
@@ -2,31 +2,8 @@
 <robot xmlns:xacro="http://www.ros.org/wiki/xacro">
   <xacro:macro name="wheel_gazebo" params="name">
-      <gravity>true</gravity>
-      <self_collide>false</self_collide>
-    <!--gazebo reference="${name}_link">
-      <mu1 value="100.0" />
-      <mu2 value="100.0" />
-      <kp  value="1000000.0" />
-      <kd  value="1.0" />
-      <fdir1>0 1 0</fdir1>
-      <maxContacts>1</maxContacts>
-    </gazebo-->
+    <gravity>true</gravity>
+    <self_collide>false</self_collide>
   </xacro:macro>
   <xacro:macro name="base_gazebo" params="name">
-    <gazebo reference="${name}_linkx">
-      <material>Gazebo/Grey</material>
-      <gravity>true</gravity>
-      <self_collide>false</self_collide>
-    </gazebo>
-    <gazebo reference="${name}_linky">
-      <material>Gazebo/Grey</material>
-      <gravity>true</gravity>
-      <self_collide>false</self_collide>
-    </gazebo>
-    <gazebo reference="${name}_linkz">
-      <material>Gazebo/Grey</material>
-      <gravity>true</gravity>
-      <self_collide>false</self_collide>
-    </gazebo>
     <gazebo reference="origin">
       <material>Gazebo/Grey</material>

File: robotino_description/urdf/base.urdf.xacro (robot description, xacro)
@@ -3,140 +3,5 @@
   <xacro:include filename="$(find robotino_description)/urdf/base.gazebo.xacro" />
   <xacro:include filename="$(find robotino_description)/urdf/base.transmission.xacro" />
-  <xacro:macro name="base" params="name has_8dof">
-  <!--###### IF 8 DOF the joints can be moved ######-->
-  <xacro:if value="${has_8dof}">
-  <link name="origin">
-    <inertial>
-      <mass value="10" />
-      <origin xyz="0 0 0" />
-      <inertia ixx="75.0" ixy="0.0" ixz="0.0"
-        iyy="75.0" iyz="0.0"
-        izz="75.0" />
-    </inertial>
-  </link>
-   <joint name="origin_joint" type="prismatic">
-    <parent link="origin"/>
-    <child link="${name}_link"/>
-    <origin xyz="0 0 0" rpy="0 0 0" />
-    <axis xyz="1 0 0" />
-    <limit upper="20" lower="-20" effort="190" velocity="30" />
-   </joint>
-   <link name="${name}_link">
-    <inertial>
-      <mass value="10" />
-      <origin xyz="0 0 0" />
-      <inertia ixx="75.0" ixy="0.0" ixz="0.0"
-       iyy="75.0" iyz="0.0"
-       izz="75.0" />
-    </inertial>
-   </link>
-   <joint name="${name}_jointx" type="prismatic">
-    <parent link="origin"/>
-    <child link="${name}_linkx"/>
-    <origin xyz="0 0 0" rpy="0 0 0" />
-    <axis xyz="1 0 0" />
-    <limit upper="20" lower="-20" effort="0" velocity="0" />
-    <dynamics damping="1000.0" friction="1000.0"/>
-    <safety_controller k_velocity="10" k_position="15" soft_lower_limit="-10.0" soft_upper_limit="10.0" />
-   </joint>
-   <joints_transmission name="base_jointx" />
-   <joint name="${name}_jointy" type="prismatic">
-    <parent link="${name}_linkx"/>
-    <child link="${name}_linky"/>
-    <origin xyz="0 0 0" rpy="0 0 0" />
-    <axis xyz="0 1 0" />
-    <limit upper="20" lower="-20" effort="0" velocity="0" />
-    <dynamics damping="1000.0" friction="1000.0"/>
-    <safety_controller k_velocity="10" k_position="15" soft_lower_limit="-10.0" soft_upper_limit="10.0" />
-   </joint>
-   <joints_transmission name="base_jointy" />
-   <joint name="${name}_jointz" type="revolute">
-    <parent link="${name}_linky"/>
-    <child link="${name}_linkz"/>
-    <origin xyz="0 0 0" rpy="0 0 0" />
-    <axis xyz="0 0 1" />
-    <limit upper="3.14" lower="-3.14" effort="0" velocity="0" />
-    <dynamics damping="1000.0" friction="1000.0"/>
-    <safety_controller k_velocity="10" k_position="15" soft_lower_limit="-3.14" soft_upper_limit="3.14" />
-   </joint>
-   <joints_transmission name="base_jointz" />
-  <link name="${name}_linkx">
-   <inertial>
-    <mass value="0.01"/>
-    <origin xyz="0 0 0"/>
-    <inertia ixx="0.001" ixy="0.0" ixz="0.0" iyy="0.001" iyz="0.0" izz="0.001" />
-   </inertial>
-   </link>
-  <link name="${name}_linky">
-   <inertial>
-    <mass value="0.01"/>
-    <origin xyz="0 0 0"/>
-    <inertia ixx="0.001" ixy="0.0" ixz="0.0" iyy="0.001" iyz="0.0" izz="0.001" />
-   </inertial>
-   </link>
-  <link name="${name}_linkz">
-   <inertial>
-    <mass value="0.01"/>
-    <origin xyz="0 0 0"/>
-    <inertia ixx="0.001" ixy="0.0" ixz="0.0" iyy="0.001" iyz="0.0" izz="0.001" />
-   </inertial>
-   </link>
-   <joint name="${name}_body_joint" type="fixed">
-    <parent link="${name}_linkz"/>
-    <child link="${name}_body_link"/>
-    <origin xyz="0 0 0" rpy="0 0 0" />
-   </joint>
-  <link name="${name}_body_link">
-    <inertial>
-      <mass value="10" />
-      <origin xyz="0 0 0" />
-      <inertia ixx="75.0" ixy="0.0" ixz="0.0"
-       iyy="75.0" iyz="0.0"
-       izz="75.0" />
-    </inertial>
-    <visual>
-      <origin xyz="0.01 0 0" rpy="0 0 0"/>
-      <geometry>
-       <mesh filename="package://robotino_description/meshes/RobotinoBody.dae"/>
-      </geometry>
-    </visual>
-    <collision>
-      <origin xyz="0.01 0 0.12" rpy="0 0 0"/>
-      <geometry>
-       <cylinder length="0.24" radius="0.23"/>
-      </geometry>
-    </collision>
-   </link>
-   <base_gazebo name="base" />
-  <gazebo>
-    <plugin name="base_controller" filename="libgazebo_ros_planar_move.so">
-      <commandTopic>cmd_vel</commandTopic>
-      <odometryTopic>odom</odometryTopic>
-      <odometryFrame>odom</odometryFrame>
-      <odometryRate>20.0</odometryRate>
-      <robotBaseFrame>origin</robotBaseFrame>
-    </plugin>
-  </gazebo>
-   <wheel name="wheel0" parent="base_linkz">
-    <origin xyz="0.095 0.14 0.02" rpy="0 0 ${M_PI/3}"/>
-    <axis xyz="-1 0 0"/>
-   </wheel>
-   <wheel_transmission name="wheel0" />
-   <wheel_gazebo name="wheel0" />
-   <wheel name="wheel1" parent="base_linkz">
-    <origin xyz="-0.16 0 0.02" rpy="0 0 0"/>
-    <axis xyz="1 0 0"/>
-   </wheel>
-   <wheel_transmission name="wheel1" />
-   <wheel_gazebo name="wheel1" />
-   <wheel name="wheel2" parent="base_linkz">
-    <origin xyz="0.105 -0.15 0.02" rpy="0 0 -${M_PI/3}"/>
-    <axis xyz="-1 0 0"/>
-   </wheel>
-   <wheel_transmission name="wheel2" />
-   <wheel_gazebo name="wheel2" />
-  </xacro:if>
- <!--###### ELSE the joints are fixed ######-->
-  <xacro:unless value="${has_8dof}">
+  <xacro:macro name="base" params="name">
   <link name="${name}_link" />
    <joint name="${name}_body_joint" type="fixed">
@@ -194,5 +59,4 @@
    <wheel_transmission name="wheel2" />
    <wheel_gazebo name="wheel2" />
-  </xacro:unless>
   </xacro:macro>
   <!-- WHEEL -->
