Commit message: updates

File: robotino_description/urdf/hokuyo.urdf.xacro (robot description, xacro)
@@ -22,5 +22,5 @@
       </visual>
       <collision>
-        <origin xyz="0 0 ${HOKUYO_LENGTH/2}" rpy="0 0 0" />
+        <origin xyz="0.0 0 ${HOKUYO_LENGTH}" rpy="0 0 0" />
         <geometry>
           <cylinder radius="${HOKUYO_RADIUS}" length="${HOKUYO_LENGTH}" />

Commit message: some misalignment

File: robotino_description/urdf/hokuyo.urdf.xacro (robot description, xacro)
@@ -22,5 +22,5 @@
       </visual>
       <collision>
-        <origin xyz="0.0 0 ${HOKUYO_LENGTH}" rpy="0 0 0" />
+        <origin xyz="0 0 ${HOKUYO_LENGTH/2}" rpy="0 0 0" />
         <geometry>
           <cylinder radius="${HOKUYO_RADIUS}" length="${HOKUYO_LENGTH}" />
