Commit message: updated urdf

File: robotino_description/urdf/arm.urdf.xacro (robot description, xacro)
@@ -1,29 +1,17 @@
 <?xml version="1.0"?>
 <robot xmlns:xacro="http://wiki.ros.org/xacro">
-  <xacro:macro name="arm">
-    <link name="base">
+  <xacro:macro name="arm" params="parent *origin name">
+    <joint name="${name}base_joint" type="revolute">
+      <parent link="${parent}"/>
+      <child link="${name}link0"/>
+      <axis xyz="0 0 1" />
+      <insert_block name="origin" />
+      <limit upper="1.7" lower="-1.7" effort="160" velocity="30" />
+    </joint>
+    <link name="${name}link0">
       <xacro:default_inertial/>
       <visual>
         <geometry>
-          <box size="0.04096 0.0473 0.105" />
-        </geometry>
-        <material name="white">
-          <color rgba="1 1 1 1"/>
-        </material>
-        <origin rpy="0 0 0" xyz="0 0 0.0525"/>
-      </visual>
-    </link>
-    <joint name="baserot" type="revolute">
-      <parent link="base"/>
-      <child link="motor1"/>
-      <axis xyz="0 0 1" />
-      <origin xyz="0.0 -0.01591 0.140" rpy="0 0 0" />
-      <limit upper="1.7" lower="-1.7" effort="160" velocity="30" />
-    </joint>
-    <link name="motor1">
-      <xacro:default_inertial/>
-      <visual>
-        <geometry>
-          <mesh filename="package://robotino_description/meshes/arm/motor1.stl"/>
+          <mesh filename="package://robotino_description/meshes/arm/link0.stl"/>
         </geometry>
         <material name="white">
@@ -35,16 +23,16 @@
         <origin rpy="0 0 0" xyz="0 0 0."/>
         <geometry>
-          <mesh filename="package://robotino_description/meshes/arm/motor1_collision.stl"/>
+          <mesh filename="package://robotino_description/meshes/arm/link0_collision.stl"/>
         </geometry>
       </collision>
     </link>
-    <joint name="joint1" type="revolute">
-      <parent link="motor1"/>
-      <child link="link1"/>
+    <joint name="${name}joint1" type="revolute">
+      <parent link="${name}link0"/>
+      <child link="${name}link1"/>
       <origin xyz="0.0 0.0 0.0" rpy="0 0 0" />
       <axis xyz="0 1 0" />
       <limit upper="1.9" lower="-1.9" effort="190" velocity="30" />
     </joint>
-    <link name="link1">
+    <link name="${name}link1">
       <xacro:default_inertial/>
       <visual>
@@ -62,11 +50,11 @@
       </collision>
     </link>
-    <gazebo reference="link1">
+    <gazebo reference="${name}link1">
         <material>Gazebo/White</material>
     </gazebo>
-    <joint name="joint2" type="revolute">
-      <parent link="link1"/>
+    <joint name="${name}joint2" type="revolute">
+      <parent link="${name}link1"/>
       <child link="motor2"/>
-      <origin xyz="0.0 0.09 0.28" rpy="0 0 0" />
+      <origin xyz="0.0 0.0 0.25" rpy="0 0 0" />
       <axis xyz="0 1 0" />
       <limit upper="1.9" lower="-1.9" effort="190" velocity="30" />
@@ -84,8 +72,8 @@
     <joint name="fixed_motor2_link2" type="fixed">
       <parent link="motor2"/>
-      <child link="link2"/>
+      <child link="${name}link2"/>
       <origin xyz="0.0 0.098 0.027" rpy="0 0 0" />
     </joint>
-    <link name="link2">
+    <link name="${name}link2">
       <xacro:default_inertial/>
       <visual>
@@ -103,15 +91,15 @@
       </collision>
     </link>
-    <gazebo reference="link2">
+    <gazebo reference="${name}link2">
       <material>Gazebo/White</material>
     </gazebo>
-    <joint name="joint3" type="revolute">
-      <parent link="link2"/>
-      <child link="link3"/>
+    <joint name="${name}joint3" type="revolute">
+      <parent link="${name}link2"/>
+      <child link="${name}link3"/>
       <origin xyz="0.0 0.0 0.13" rpy="0 0 0" />
       <axis xyz="0 0 1" />
       <limit upper="1.7" lower="-1.7" effort="190" velocity="30" />
     </joint>
-    <link name="link3">
+    <link name="${name}link3">
       <xacro:default_inertial/>
       <visual>
@@ -129,15 +117,15 @@
       </collision>
     </link>
-    <gazebo reference="link3">
+    <gazebo reference="${name}link3">
       <material>Gazebo/White</material>
     </gazebo>
-    <joint name="joint4" type="revolute">
-      <parent link="link3"/>
-      <child link="link4"/>
+    <joint name="${name}joint4" type="revolute">
+      <parent link="${name}link3"/>
+      <child link="${name}link4"/>
       <origin xyz="0.0 -0.053 0.065" rpy="0 0 0" />
       <axis xyz="0 1 0" />
       <limit upper="1.7" lower="-1.7" effort="160" velocity="30" />
     </joint>
-    <link name="link4">
+    <link name="${name}link4">
       <xacro:default_inertial/>
       <visual>
@@ -155,18 +143,18 @@
       </collision>
     </link>
-    <gazebo reference="link4">
+    <gazebo reference="${name}link4">
       <material>Gazebo/White</material>
     </gazebo>
-    <joint name="joint5" type="revolute">
-      <parent link="link4"/>
-      <child link="link5"/>
+    <joint name="${name}joint5" type="revolute">
+      <parent link="${name}link4"/>
+      <child link="${name}link5"/>
       <origin xyz="0.0 -0.027 0.035" rpy="0 0 0" />
       <axis xyz="0 0 1" />
       <limit upper="1.7" lower="-1.7" effort="160" velocity="30" />
     </joint>
-    <link name="link5">
+    <link name="${name}link5">
       <xacro:default_inertial/>
     </link>
-    <gazebo reference="link5">
+    <gazebo reference="${name}link5">
       <material>Gazebo/White</material>
     </gazebo>
@@ -176,13 +164,19 @@
   <xacro:arm_SimpleTransmission number="4"></xacro:arm_SimpleTransmission>
   <xacro:arm_SimpleTransmission number="5"></xacro:arm_SimpleTransmission>
-  <xacro:arm_SimpleTransmission number="6"></xacro:arm_SimpleTransmission>
-  <xacro:arm_SimpleTransmission number="7"></xacro:arm_SimpleTransmission>
+    <transmission name="${name}base_trans">
+      <type>transmission_interface/SimpleTransmission</type>
+      <joint name="${name}base_joint">
+        <hardwareInterface>PositionJointInterface</hardwareInterface>
+      </joint>
+      <actuator name="${name}base_motor">
+        <mechanicalReduction>1</mechanicalReduction>
+      </actuator>
+    </transmission>
   </xacro:macro>
   <xacro:macro name="arm_SimpleTransmission" params="number">
     <transmission name="arm_${number}_trans">
       <type>transmission_interface/SimpleTransmission</type>
-      <joint name="joint${number}">
+      <joint name="${name}joint${number}">
         <hardwareInterface>PositionJointInterface</hardwareInterface>
-        <hardwareInterface>VelocityJointInterface</hardwareInterface>
       </joint>
       <actuator name="arm_${number}_motor">

Commit message: default inertia values for hand links

File: robotino_description/urdf/arm.urdf.xacro (robot description, xacro)
@@ -97,5 +97,5 @@
       <parent link="${name}link2"/>
       <child link="${name}link3"/>
-      <origin xyz="0.0 0.0 0.13" rpy="0 0 0" />
+      <origin xyz="0.0 0.0 0.158" rpy="0 0 0" />
       <axis xyz="0 0 1" />
       <limit upper="1.7" lower="-1.7" effort="190" velocity="30" />
@@ -123,5 +123,5 @@
       <parent link="${name}link3"/>
       <child link="${name}link4"/>
-      <origin xyz="0.0 -0.053 0.065" rpy="0 0 0" />
+      <origin xyz="0.0 -0.057 0.065" rpy="0 0 0" />
       <axis xyz="0 1 0" />
       <limit upper="1.7" lower="-1.7" effort="160" velocity="30" />

Commit message: clean and review arm link names

File: robotino_description/urdf/arm.urdf.xacro (robot description, xacro)
@@ -4,10 +4,10 @@
     <joint name="${name}base_joint" type="revolute">
       <parent link="${parent}"/>
-      <child link="${name}link0"/>
+      <child link="${name}base_link"/>
       <axis xyz="0 0 1" />
       <insert_block name="origin" />
       <limit upper="1.7" lower="-1.7" effort="160" velocity="30" />
     </joint>
-    <link name="${name}link0">
+    <link name="${name}base_link">
       <xacro:default_inertial/>
       <visual>
@@ -28,5 +28,5 @@
     </link>
     <joint name="${name}joint1" type="revolute">
-      <parent link="${name}link0"/>
+      <parent link="${name}base_link"/>
       <child link="${name}link1"/>
       <origin xyz="0.0 0.0 0.0" rpy="0 0 0" />
@@ -55,10 +55,10 @@
     <joint name="${name}joint2" type="revolute">
       <parent link="${name}link1"/>
-      <child link="motor2"/>
+      <child link="${name}motor2"/>
       <origin xyz="0.0 0.0 0.25" rpy="0 0 0" />
       <axis xyz="0 1 0" />
       <limit upper="1.9" lower="-1.9" effort="190" velocity="30" />
     </joint>
-    <link name="motor2">
+    <link name="${name}motor2">
       <xacro:default_inertial/>
       <visual>
@@ -71,5 +71,5 @@
     </link>
     <joint name="fixed_motor2_link2" type="fixed">
-      <parent link="motor2"/>
+      <parent link="${name}motor2"/>
       <child link="${name}link2"/>
       <origin xyz="0.0 0.098 0.027" rpy="0 0 0" />

Commit message: 8 dof description

File: robotino_description/urdf/arm.urdf.xacro (robot description, xacro)
@@ -2,10 +2,8 @@
 <robot xmlns:xacro="http://wiki.ros.org/xacro">
   <xacro:macro name="arm" params="parent *origin name">
-    <joint name="${name}base_joint" type="revolute">
+    <joint name="${name}base_joint" type="fixed">
       <parent link="${parent}"/>
       <child link="${name}link0"/>
-      <axis xyz="0 0 1" />
       <insert_block name="origin" />
-      <limit upper="1.7" lower="-1.7" effort="160" velocity="30" />
     </joint>
     <link name="${name}link0">

Commit message: changes in robot limit tested working

File: robotino_description/urdf/arm.urdf.xacro (robot description, xacro)
@@ -31,5 +31,5 @@
       <origin xyz="0.0 0.0 0.0" rpy="0 0 0" />
       <axis xyz="0 1 0" />
-      <limit upper="1.9" lower="-1.9" effort="190" velocity="30" />
+      <limit upper="1.5" lower="-1.2" effort="190" velocity="30" />
     </joint>
     <link name="${name}link1">
@@ -57,5 +57,5 @@
       <origin xyz="0.0 0.0 0.25" rpy="0 0 0" />
       <axis xyz="0 1 0" />
-      <limit upper="1.9" lower="-1.9" effort="190" velocity="30" />
+      <limit upper="2.3" lower="-1.7" effort="190" velocity="30" />
     </joint>
     <link name="${name}motor2">
@@ -98,5 +98,5 @@
       <origin xyz="0.0 0.0 0.158" rpy="0 0 0" />
       <axis xyz="0 0 1" />
-      <limit upper="1.7" lower="-1.7" effort="190" velocity="30" />
+      <limit upper="1.8" lower="-1.8" effort="190" velocity="30" />
     </joint>
     <link name="${name}link3">
@@ -124,5 +124,5 @@
       <origin xyz="0.0 -0.057 0.065" rpy="0 0 0" />
       <axis xyz="0 1 0" />
-      <limit upper="1.7" lower="-1.7" effort="160" velocity="30" />
+      <limit upper="1.9" lower="-1.9" effort="160" velocity="30" />
     </joint>
     <link name="${name}link4">
@@ -150,5 +150,5 @@
       <origin xyz="0.0 -0.027 0.035" rpy="0 0 0" />
       <axis xyz="0 0 1" />
-      <limit upper="1.7" lower="-1.7" effort="160" velocity="30" />
+      <limit upper="2.9" lower="-2.9" effort="160" velocity="30" />
     </joint>
     <link name="${name}link5">

File: robotino_description/urdf/base.urdf.xacro (robot description, xacro)
@@ -20,5 +20,5 @@
     <origin xyz="0 0 0" rpy="0 0 0" />
     <axis xyz="1 0 0" />
-    <limit upper="10" lower="-10" effort="190" velocity="30" />
+    <limit upper="20" lower="-20" effort="190" velocity="30" />
    </joint>
    <link name="${name}_link">
@@ -36,7 +36,7 @@
     <origin xyz="0 0 0" rpy="0 0 0" />
     <axis xyz="1 0 0" />
-    <limit upper="10" lower="-10" effort="0" velocity="0" />
+    <limit upper="20" lower="-20" effort="0" velocity="0" />
     <dynamics damping="1000.0" friction="1000.0"/>
-    <safety_controller k_velocity="10" k_position="15" soft_lower_limit="-2.0" soft_upper_limit="0.5" />
+    <safety_controller k_velocity="10" k_position="15" soft_lower_limit="-10.0" soft_upper_limit="10.0" />
    </joint>
    <joints_transmission name="base_jointx" />
@@ -46,7 +46,7 @@
     <origin xyz="0 0 0" rpy="0 0 0" />
     <axis xyz="0 1 0" />
-    <limit upper="10" lower="-10" effort="0" velocity="0" />
+    <limit upper="20" lower="-20" effort="0" velocity="0" />
     <dynamics damping="1000.0" friction="1000.0"/>
-    <safety_controller k_velocity="10" k_position="15" soft_lower_limit="-2.0" soft_upper_limit="0.5" />
+    <safety_controller k_velocity="10" k_position="15" soft_lower_limit="-10.0" soft_upper_limit="10.0" />
    </joint>
    <joints_transmission name="base_jointy" />
@@ -58,5 +58,5 @@
     <limit upper="3.14" lower="-3.14" effort="0" velocity="0" />
     <dynamics damping="1000.0" friction="1000.0"/>
-    <safety_controller k_velocity="10" k_position="15" soft_lower_limit="-2.0" soft_upper_limit="0.5" />
+    <safety_controller k_velocity="10" k_position="15" soft_lower_limit="-3.14" soft_upper_limit="3.14" />
    </joint>
    <joints_transmission name="base_jointz" />

Commit message: Modifications from year3 review

File: robotino_description/urdf/arm.urdf.xacro (robot description, xacro)
@@ -31,5 +31,5 @@
       <origin xyz="0.0 0.0 0.0" rpy="0 0 0" />
       <axis xyz="0 1 0" />
-      <limit upper="1.5" lower="-1.2" effort="190" velocity="30" />
+      <limit upper="1.5" lower="-0.3" effort="190" velocity="30" />
     </joint>
     <link name="${name}link1">

File: robotino_description/urdf/base.urdf.xacro (robot description, xacro)
@@ -160,9 +160,15 @@
     </visual>
     <collision>
+      <origin xyz="0.01 0 0.12" rpy="0 0 0"/>
+      <geometry>
+       <cylinder length="0.24" radius="0.23"/>
+      </geometry>
+    </collision>
+    <!--collision>
       <origin xyz="0.01 0 0" rpy="0 0 0"/>
       <geometry>
        <mesh filename="package://robotino_description/meshes/RobotinoBody.stl"/>
       </geometry>
-    </collision>
+    </collision-->
    </link>
    <base_gazebo name="base" />

Commit message: udpated joint limits for folding the arm

File: robotino_description/urdf/arm.urdf.xacro (robot description, xacro)
@@ -57,5 +57,5 @@
       <origin xyz="0.0 0.0 0.25" rpy="0 0 0" />
       <axis xyz="0 1 0" />
-      <limit upper="2.3" lower="-1.7" effort="190" velocity="30" />
+      <limit upper="2.6" lower="-1.7" effort="190" velocity="30" />
     </joint>
     <link name="${name}motor2">
@@ -124,5 +124,5 @@
       <origin xyz="0.0 -0.057 0.065" rpy="0 0 0" />
       <axis xyz="0 1 0" />
-      <limit upper="1.9" lower="-1.9" effort="160" velocity="30" />
+      <limit upper="2.4" lower="-2.4" effort="160" velocity="30" />
     </joint>
     <link name="${name}link4">

Commit message: review motor directions for the arm

File: robotino_description/urdf/arm.urdf.xacro (robot description, xacro)
@@ -30,5 +30,5 @@
       <child link="${name}link1"/>
       <origin xyz="0.0 0.0 0.0" rpy="0 0 0" />
-      <axis xyz="0 1 0" />
+      <axis xyz="0 -1 0" />
       <limit upper="1.5" lower="-1.2" effort="190" velocity="30" />
     </joint>
@@ -123,5 +123,5 @@
       <child link="${name}link4"/>
       <origin xyz="0.0 -0.057 0.065" rpy="0 0 0" />
-      <axis xyz="0 1 0" />
+      <axis xyz="0 -1 0" />
       <limit upper="2.4" lower="-2.4" effort="160" velocity="30" />
     </joint>

Commit message: updated velocities and effrots

File: robotino_description/urdf/arm.urdf.xacro (robot description, xacro)
@@ -31,5 +31,5 @@
       <origin xyz="0.0 0.0 0.0" rpy="0 0 0" />
       <axis xyz="0 -1 0" />
-      <limit upper="1.5" lower="-1.2" effort="190" velocity="30" />
+      <limit upper="1.5" lower="-1.2" effort="90" velocity="0.7" />
     </joint>
     <link name="${name}link1">
@@ -57,5 +57,5 @@
       <origin xyz="0.0 0.0 0.25" rpy="0 0 0" />
       <axis xyz="0 1 0" />
-      <limit upper="2.6" lower="-1.7" effort="190" velocity="30" />
+      <limit upper="2.6" lower="-1.7" effort="90" velocity="0.7" />
     </joint>
     <link name="${name}motor2">
@@ -98,5 +98,5 @@
       <origin xyz="0.0 0.0 0.158" rpy="0 0 0" />
       <axis xyz="0 0 1" />
-      <limit upper="1.8" lower="-1.8" effort="190" velocity="30" />
+      <limit upper="1.8" lower="-1.8" effort="90" velocity="0.7" />
     </joint>
     <link name="${name}link3">
@@ -124,5 +124,5 @@
       <origin xyz="0.0 -0.057 0.065" rpy="0 0 0" />
       <axis xyz="0 -1 0" />
-      <limit upper="2.4" lower="-2.4" effort="160" velocity="30" />
+      <limit upper="2.4" lower="-2.4" effort="90" velocity="0.7" />
     </joint>
     <link name="${name}link4">
@@ -150,5 +150,5 @@
       <origin xyz="0.0 -0.027 0.035" rpy="0 0 0" />
       <axis xyz="0 0 1" />
-      <limit upper="2.9" lower="-2.9" effort="160" velocity="30" />
+      <limit upper="2.9" lower="-2.9" effort="90" velocity="0.7" />
     </joint>
     <link name="${name}link5">

File: robotino_description/urdf/base.urdf.xacro (robot description, xacro)
@@ -35,5 +35,5 @@
     <origin xyz="0 0 0" rpy="0 0 0" />
     <axis xyz="1 0 0" />
-    <limit upper="20" lower="-20" effort="0" velocity="0" />
+    <limit upper="20" lower="-20" effort="90" velocity="0.3" />
     <dynamics damping="1000.0" friction="1000.0"/>
     <safety_controller k_velocity="10" k_position="15" soft_lower_limit="-10.0" soft_upper_limit="10.0" />
@@ -45,5 +45,5 @@
     <origin xyz="0 0 0" rpy="0 0 0" />
     <axis xyz="0 1 0" />
-    <limit upper="20" lower="-20" effort="0" velocity="0" />
+    <limit upper="20" lower="-20" effort="90" velocity="0.3" />
     <dynamics damping="1000.0" friction="1000.0"/>
     <safety_controller k_velocity="10" k_position="15" soft_lower_limit="-10.0" soft_upper_limit="10.0" />
@@ -55,5 +55,5 @@
     <origin xyz="0 0 0" rpy="0 0 0" />
     <axis xyz="0 0 1" />
-    <limit upper="3.14" lower="-3.14" effort="0" velocity="0" />
+    <limit upper="3.14" lower="-3.14" effort="90" velocity="0.7" />
     <dynamics damping="1000.0" friction="1000.0"/>
     <safety_controller k_velocity="10" k_position="15" soft_lower_limit="-3.14" soft_upper_limit="3.14" />

Commit message: joint directions review

File: robotino_description/urdf/arm.urdf.xacro (robot description, xacro)
@@ -30,5 +30,5 @@
       <child link="${name}link1"/>
       <origin xyz="0.0 0.0 0.0" rpy="0 0 0" />
-      <axis xyz="0 -1 0" />
+      <axis xyz="0 1 0" />
       <limit upper="1.5" lower="-1.2" effort="90" velocity="0.7" />
     </joint>
@@ -123,6 +123,6 @@
       <child link="${name}link4"/>
       <origin xyz="0.0 -0.057 0.065" rpy="0 0 0" />
+      <axis xyz="0 1 0" />
       <limit upper="2.4" lower="-2.4" effort="90" velocity="0.7" />
-      <axis xyz="0 1 0" />
     </joint>
     <link name="${name}link4">

Commit message: revert motor directions

File: robotino_description/urdf/arm.urdf.xacro (robot description, xacro)
@@ -30,5 +30,5 @@
       <child link="${name}link1"/>
       <origin xyz="0.0 0.0 0.0" rpy="0 0 0" />
-      <axis xyz="0 1 0" />
+      <axis xyz="0 -1 0" />
       <limit upper="1.5" lower="-1.2" effort="90" velocity="0.7" />
     </joint>
@@ -123,5 +123,5 @@
       <child link="${name}link4"/>
       <origin xyz="0.0 -0.057 0.065" rpy="0 0 0" />
-      <axis xyz="0 1 0" />
+      <axis xyz="0 -1 0" />
       <limit upper="2.4" lower="-2.4" effort="90" velocity="0.7" />
     </joint>
