Commit message: base 8 dof

File: robotino_description/urdf/base.urdf.xacro (robot description, xacro)
@@ -149,3 +149,15 @@
     </transmission>
   </xacro:macro>
+  <xacro:macro name="joints_transmission" params="name">
+    <transmission name="${name}_trans">
+      <type>transmission_interface/SimpleTransmission</type>
+      <joint name="${name}" >
+        <hardwareInterface>VelocityJointInterface</hardwareInterface>
+      </joint>
+      <actuator name="${name}_motor">
+        <hardwareInterface>VelocityJointInterface</hardwareInterface>
+        <mechanicalReduction>${ 624/35 * 80/18}</mechanicalReduction>
+      </actuator>
+    </transmission>
+  </xacro:macro>
 </root>

Commit message: made navigation and planning to work in parallel

File: robotino_description/urdf/base.urdf.xacro (robot description, xacro)
@@ -3,5 +3,12 @@
   <xacro:include filename="$(find robotino_description)/urdf/gazebo.urdf.xacro" />
   <xacro:macro name="base" params="name">
-   <link name="${name}_link">
+   <joint name="origin_joint" type="prismatic">
+	  <parent link="origin"/>
+      <child link="${name}_link"/>
+      <origin xyz="0 0 0" rpy="0 0 0" />
+      <axis xyz="1 0 0" />
+      <limit upper="10" lower="-10" effort="190" velocity="30" />
+    </joint>
+    <link name="${name}_link">
       <inertial>
         <mass value="10" />
@@ -13,5 +20,6 @@
     </link>
     <joint name="${name}_jointx" type="prismatic">
-      <parent link="${name}_link"/>
+<!--      <parent link="${name}_link"/>-->
+	  <parent link="origin"/>
       <child link="${name}_linkx"/>
       <origin xyz="0 0 0" rpy="0 0 0" />

Commit message: addapted base to 8 dof modus

File: robotino_description/urdf/base.urdf.xacro (robot description, xacro)
@@ -1,171 +1,203 @@
 <?xml version="1.0"?>
 <root xmlns:xacro="http://www.ros.org/wiki/xacro">
-  <xacro:include filename="$(find robotino_description)/urdf/gazebo.urdf.xacro" />
-  <xacro:macro name="base" params="name">
-   <joint name="origin_joint" type="prismatic">
-	  <parent link="origin"/>
-      <child link="${name}_link"/>
-      <origin xyz="0 0 0" rpy="0 0 0" />
-      <axis xyz="1 0 0" />
-      <limit upper="10" lower="-10" effort="190" velocity="30" />
-    </joint>
-    <link name="${name}_link">
-      <inertial>
-        <mass value="10" />
-        <origin xyz="0 0 0" />
-        <inertia ixx="75.0" ixy="0.0" ixz="0.0"
-          iyy="75.0" iyz="0.0"
-          izz="75.0" />
-      </inertial>
-    </link>
-    <joint name="${name}_jointx" type="prismatic">
-<!--      <parent link="${name}_link"/>-->
-	  <parent link="origin"/>
-      <child link="${name}_linkx"/>
-      <origin xyz="0 0 0" rpy="0 0 0" />
-      <axis xyz="1 0 0" />
-      <limit upper="10" lower="-10" effort="190" velocity="30" />
-    </joint>
-   <link name="${name}_linkx">
-      <inertial>
-        <mass value="10" />
-        <origin xyz="0 0 0" />
-        <inertia ixx="75.0" ixy="0.0" ixz="0.0"
-          iyy="75.0" iyz="0.0"
-          izz="75.0" />
-      </inertial>
-    </link>
-    <joint name="${name}_jointy" type="prismatic">
-      <parent link="${name}_linkx"/>
-      <child link="${name}_linky"/>
-      <origin xyz="0 0 0" rpy="0 0 0" />
-      <axis xyz="0 1 0" />
-      <limit upper="10" lower="-10" effort="190" velocity="30" />
-    </joint>
-   <link name="${name}_linky">
-      <inertial>
-        <mass value="10" />
-        <origin xyz="0 0 0" />
-        <inertia ixx="75.0" ixy="0.0" ixz="0.0"
-          iyy="75.0" iyz="0.0"
-          izz="75.0" />
-      </inertial>
-    </link>
-    <joint name="${name}_jointz" type="revolute">
-      <parent link="${name}_linky"/>
-      <child link="${name}_linkz"/>
-      <origin xyz="0 0 0" rpy="0 0 0" />
-      <axis xyz="0 0 1" />
-      <limit upper="3.14" lower="-3.14" effort="190" velocity="30" />
-    </joint>
-   <link name="${name}_linkz">
-      <inertial>
-        <mass value="10" />
-        <origin xyz="0 0 0" />
-        <inertia ixx="75.0" ixy="0.0" ixz="0.0"
-          iyy="75.0" iyz="0.0"
-          izz="75.0" />
-      </inertial>
-    </link>
-    <joint name="${name}_body_joint" type="fixed">
-      <parent link="${name}_linkz"/>
-      <child link="${name}_body_link"/>
-      <origin xyz="0 0 0" rpy="0 0 0" />
-    </joint>
-   <link name="${name}_body_link">
-      <inertial>
-        <mass value="10" />
-        <origin xyz="0 0 0" />
-        <inertia ixx="75.0" ixy="0.0" ixz="0.0"
-          iyy="75.0" iyz="0.0"
-          izz="75.0" />
-      </inertial>
-      <visual>
-        <origin xyz="0.01 0 0" rpy="0 0 0"/>
-        <geometry>
-          <mesh filename="package://robotino_description/meshes/RobotinoBody.dae"/>
-        </geometry>
-      </visual>
-      <collision>
-        <origin xyz="0.01 0 0" rpy="0 0 0"/>
-        <geometry>
-          <mesh filename="package://robotino_description/meshes/RobotinoBody.stl"/>
-        </geometry>
-      </collision>
-    </link>
-    <base_gazebo name="base" />
-    <wheel name="wheel0" parent="base_linkz">
-      <origin xyz="0.095 0.14 0.02" rpy="0 0 ${M_PI/3}"/>
-      <axis xyz="-1 0 0"/>
-    </wheel>
-    <wheel_transmission name="wheel0" />
-    <wheel_gazebo name="wheel0" />
-    <wheel name="wheel1" parent="base_linkz">
-      <origin xyz="-0.16 0 0.02" rpy="0 0 0"/>
-      <axis xyz="1 0 0"/>
-    </wheel>
-    <wheel_transmission name="wheel1" />
-    <wheel_gazebo name="wheel1" />
-    <wheel name="wheel2" parent="base_linkz">
-      <origin xyz="0.105 -0.15 0.02" rpy="0 0 -${M_PI/3}"/>
-      <axis xyz="-1 0 0"/>
-    </wheel>
-    <wheel_transmission name="wheel2" />
-    <wheel_gazebo name="wheel2" />
+  <xacro:include filename="$(find robotino_description)/urdf/base.gazebo.xacro" />
+  <xacro:include filename="$(find robotino_description)/urdf/base.transmission.xacro" />
+  <xacro:macro name="base" params="name has_8dof">
+  <link name="origin" />
+  <joint name="origin_joint" type="fixed">
+    <origin xyz="0 0 0" rpy="0 0 0"/>
+    <parent link="origin"/>
+    <child link="${name}_link"/>
+   </joint>
+   <link name="${name}_link">
+    <inertial>
+      <mass value="10" />
+      <origin xyz="0 0 0" />
+      <inertia ixx="75.0" ixy="0.0" ixz="0.0"
+       iyy="75.0" iyz="0.0"
+       izz="75.0" />
+    </inertial>
+   </link>
+  <!--###### IF 8 DOF the joints can be moved ######-->
+  <xacro:if value="${has_8dof}">
+   <joint name="${name}_jointx" type="prismatic">
+    <parent link="origin"/>
+    <child link="${name}_linkx"/>
+    <origin xyz="0 0 0" rpy="0 0 0" />
+    <axis xyz="1 0 0" />
+    <limit upper="10" lower="-10" effort="0" velocity="0" />
+    <dynamics damping="1000.0" friction="1000.0"/>
+    <safety_controller k_velocity="10" k_position="15" soft_lower_limit="-2.0" soft_upper_limit="0.5" />
+   </joint>
+   <joints_transmission name="base_jointx" />
+   <joint name="${name}_jointy" type="prismatic">
+    <parent link="${name}_linkx"/>
+    <child link="${name}_linky"/>
+    <origin xyz="0 0 0" rpy="0 0 0" />
+    <axis xyz="0 1 0" />
+    <limit upper="10" lower="-10" effort="0" velocity="0" />
+    <dynamics damping="1000.0" friction="1000.0"/>
+    <safety_controller k_velocity="10" k_position="15" soft_lower_limit="-2.0" soft_upper_limit="0.5" />
+   </joint>
+   <joints_transmission name="base_jointy" />
+   <joint name="${name}_jointz" type="revolute">
+    <parent link="${name}_linky"/>
+    <child link="${name}_linkz"/>
+    <origin xyz="0 0 0" rpy="0 0 0" />
+    <axis xyz="0 0 1" />
+    <limit upper="3.14" lower="-3.14" effort="0" velocity="0" />
+    <dynamics damping="1000.0" friction="1000.0"/>
+    <safety_controller k_velocity="10" k_position="15" soft_lower_limit="-2.0" soft_upper_limit="0.5" />
+   </joint>
+   <joints_transmission name="base_jointz" />
+  </xacro:if>
+  <!--###### ELSE the joints are fixed ######-->
+  <xacro:unless value="${has_8dof}">
+   <joint name="${name}_jointx" type="fixed">
+    <parent link="origin"/>
+    <child link="${name}_linkx"/>
+    <origin xyz="0 0 0" rpy="0 0 0" />
+   </joint>
+   <joint name="${name}_jointy" type="fixed">
+    <parent link="${name}_linkx"/>
+    <child link="${name}_linky"/>
+    <origin xyz="0 0 0" rpy="0 0 0" />
+   </joint>
+   <joint name="${name}_jointz" type="fixed">
+    <parent link="${name}_linky"/>
+    <child link="${name}_linkz"/>
+    <origin xyz="0 0 0" rpy="0 0 0" />
+   </joint>
+  </xacro:unless>
+  <link name="${name}_linkx">
+   <inertial>
+    <mass value="0.01"/>
+    <origin xyz="0 0 0"/>
+    <inertia ixx="0.001" ixy="0.0" ixz="0.0" iyy="0.001" iyz="0.0" izz="0.001" />
+   </inertial>
+   <visual>
+    <origin xyz="0 0 0" rpy="0 0 0" />
+    <geometry>
+      <box size="0.001 0.001 0.001" />
+    </geometry>
+   </visual>
+    <collision>
+      <origin xyz="0 0 0" rpy="0 0 0" />
+      <geometry>
+       <box size="0.001 0.001 0.001" />
+      </geometry>
+    </collision>
+   </link>
+  <link name="${name}_linky">
+   <inertial>
+    <mass value="0.01"/>
+    <origin xyz="0 0 0"/>
+    <inertia ixx="0.001" ixy="0.0" ixz="0.0" iyy="0.001" iyz="0.0" izz="0.001" />
+   </inertial>
+   <visual>
+    <origin xyz="0 0 0" rpy="0 0 0" />
+    <geometry>
+      <box size="0.001 0.001 0.001" />
+    </geometry>
+   </visual>
+    <collision>
+      <origin xyz="0 0 0" rpy="0 0 0" />
+      <geometry>
+       <box size="0.001 0.001 0.001" />
+      </geometry>
+    </collision>
+   </link>
+  <link name="${name}_linkz">
+   <inertial>
+    <mass value="0.01"/>
+    <origin xyz="0 0 0"/>
+    <inertia ixx="0.001" ixy="0.0" ixz="0.0" iyy="0.001" iyz="0.0" izz="0.001" />
+   </inertial>
+   <visual>
+    <origin xyz="0 0 0" rpy="0 0 0" />
+    <geometry>
+      <box size="0.001 0.001 0.001" />
+    </geometry>
+   </visual>
+    <collision>
+      <origin xyz="0 0 0" rpy="0 0 0" />
+      <geometry>
+       <box size="0.001 0.001 0.001" />
+      </geometry>
+    </collision>
+   </link>
+   <joint name="${name}_body_joint" type="fixed">
+    <parent link="${name}_linkz"/>
+    <child link="${name}_body_link"/>
+    <origin xyz="0 0 0" rpy="0 0 0" />
+   </joint>
+  <link name="${name}_body_link">
+    <inertial>
+      <mass value="10" />
+      <origin xyz="0 0 0" />
+      <inertia ixx="75.0" ixy="0.0" ixz="0.0"
+       iyy="75.0" iyz="0.0"
+       izz="75.0" />
+    </inertial>
+    <visual>
+      <origin xyz="0.01 0 0" rpy="0 0 0"/>
+      <geometry>
+       <mesh filename="package://robotino_description/meshes/RobotinoBody.dae"/>
+      </geometry>
+    </visual>
+    <collision>
+      <origin xyz="0.01 0 0" rpy="0 0 0"/>
+      <geometry>
+       <mesh filename="package://robotino_description/meshes/RobotinoBody.stl"/>
+      </geometry>
+    </collision>
+   </link>
+   <base_gazebo name="base" />
+   <wheel name="wheel0" parent="base_linkz">
+    <origin xyz="0.095 0.14 0.02" rpy="0 0 ${M_PI/3}"/>
+    <axis xyz="-1 0 0"/>
+   </wheel>
+   <wheel_transmission name="wheel0" />
+   <wheel_gazebo name="wheel0" />
+   <wheel name="wheel1" parent="base_linkz">
+    <origin xyz="-0.16 0 0.02" rpy="0 0 0"/>
+    <axis xyz="1 0 0"/>
+   </wheel>
+   <wheel_transmission name="wheel1" />
+   <wheel_gazebo name="wheel1" />
+   <wheel name="wheel2" parent="base_linkz">
+    <origin xyz="0.105 -0.15 0.02" rpy="0 0 -${M_PI/3}"/>
+    <axis xyz="-1 0 0"/>
+   </wheel>
+   <wheel_transmission name="wheel2" />
+   <wheel_gazebo name="wheel2" />
   </xacro:macro>
   <!-- WHEEL -->
   <xacro:macro name="wheel" params="parent name *origin *axis">
-    <joint name="${name}_joint" type="continuous">
-      <parent link="${parent}"/>
-      <child link="${name}_link" />
-      <insert_block name="origin" />
-      <insert_block name="axis" />
-    </joint>
-    <link name="${name}_link">
-      <inertial>
-        <mass value="0.4" />
-        <origin xyz="0 0 0" />
-        <inertia ixx="0.012411765597" ixy="-0.000711733678" ixz="0.00050272983" iyy="0.015218160428" iyz="-0.000004273467" izz="0.011763977943"/>
-      </inertial>
-      <visual>
-        <origin xyz="0 0 0" rpy="0 0 0" />
-        <geometry>
-		  <!--cylinder length="0.04" radius="0.04"/-->
-          <mesh filename="package://robotino_description/meshes/RobotinoWheel.dae" scale="${M_SCALE} ${M_SCALE} ${M_SCALE}"/>
-        </geometry>
-      </visual>
-      <collision>
-        <origin xyz="0 0 0" rpy="0 ${M_PI/2} 0" />
-        <geometry>
-          <!--mesh filename="package://robotino_description/meshes/RobotinoWheel.dae" scale="${M_SCALE} ${M_SCALE} ${M_SCALE}"/-->
-          <cylinder length="0.04" radius="0.04"/>
-        </geometry>
-      </collision>
-    </link>
-  </xacro:macro>
-  <!-- Wheel transmission   -->
-  <xacro:macro name="wheel_transmission" params="name">
-    <transmission name="${name}_trans">
-      <type>transmission_interface/SimpleTransmission</type>
-      <joint name="${name}_joint" >
-        <hardwareInterface>VelocityJointInterface</hardwareInterface>
-      </joint>
-      <actuator name="${name}_motor">
-        <hardwareInterface>VelocityJointInterface</hardwareInterface>
-        <mechanicalReduction>${ 624/35 * 80/18}</mechanicalReduction>
-      </actuator>
-    </transmission>
-  </xacro:macro>
-  <xacro:macro name="joints_transmission" params="name">
-    <transmission name="${name}_trans">
-      <type>transmission_interface/SimpleTransmission</type>
-      <joint name="${name}" >
-        <hardwareInterface>VelocityJointInterface</hardwareInterface>
-      </joint>
-      <actuator name="${name}_motor">
-        <hardwareInterface>VelocityJointInterface</hardwareInterface>
-        <mechanicalReduction>${ 624/35 * 80/18}</mechanicalReduction>
-      </actuator>
-    </transmission>
+   <joint name="${name}_joint" type="continuous">
+    <parent link="${parent}"/>
+    <child link="${name}_link" />
+    <insert_block name="origin" />
+    <insert_block name="axis" />
+   </joint>
+   <link name="${name}_link">
+    <inertial>
+      <mass value="0.4" />
+      <origin xyz="0 0 0" />
+      <inertia ixx="0.012411765597" ixy="-0.000711733678" ixz="0.00050272983" iyy="0.015218160428" iyz="-0.000004273467" izz="0.011763977943"/>
+    </inertial>
+    <visual>
+      <origin xyz="0 0 0" rpy="0 0 0" />
+      <geometry>
+       <mesh filename="package://robotino_description/meshes/RobotinoWheel.dae" scale="${M_SCALE} ${M_SCALE} ${M_SCALE}"/>
+      </geometry>
+    </visual>
+    <collision>
+      <origin xyz="0 0 0" rpy="0 ${M_PI/2} 0" />
+      <geometry>
+       <cylinder length="0.04" radius="0.04"/>
+      </geometry>
+    </collision>
+   </link>
   </xacro:macro>
 </root>

Commit message: test model

File: robotino_description/urdf/base.urdf.xacro (robot description, xacro)
@@ -6,9 +6,10 @@
   <!--###### IF 8 DOF the joints can be moved ######-->
   <xacro:if value="${has_8dof}">
-  <link name="origin" />
-  <joint name="origin_joint" type="fixed">
-    <origin xyz="0 0 0" rpy="0 0 0"/>
+   <joint name="origin_joint" type="prismatic">
     <parent link="origin"/>
     <child link="${name}_link"/>
+    <origin xyz="0 0 0" rpy="0 0 0" />
+    <axis xyz="1 0 0" />
+    <limit upper="10" lower="-10" effort="190" velocity="30" />
    </joint>
    <link name="${name}_link">

Commit message: removed collision and visual parts of virtual joints

File: robotino_description/urdf/base.urdf.xacro (robot description, xacro)
@@ -58,16 +58,4 @@
     <inertia ixx="0.001" ixy="0.0" ixz="0.0" iyy="0.001" iyz="0.0" izz="0.001" />
    </inertial>
-   <visual>
-    <origin xyz="0 0 0" rpy="0 0 0" />
-    <geometry>
-      <box size="0.001 0.001 0.001" />
-    </geometry>
-   </visual>
-    <collision>
-      <origin xyz="0 0 0" rpy="0 0 0" />
-      <geometry>
-       <box size="0.001 0.001 0.001" />
-      </geometry>
-    </collision>
    </link>
   <link name="${name}_linky">
@@ -77,16 +65,4 @@
     <inertia ixx="0.001" ixy="0.0" ixz="0.0" iyy="0.001" iyz="0.0" izz="0.001" />
    </inertial>
-   <visual>
-    <origin xyz="0 0 0" rpy="0 0 0" />
-    <geometry>
-      <box size="0.001 0.001 0.001" />
-    </geometry>
-   </visual>
-    <collision>
-      <origin xyz="0 0 0" rpy="0 0 0" />
-      <geometry>
-       <box size="0.001 0.001 0.001" />
-      </geometry>
-    </collision>
    </link>
   <link name="${name}_linkz">
@@ -96,16 +72,4 @@
     <inertia ixx="0.001" ixy="0.0" ixz="0.0" iyy="0.001" iyz="0.0" izz="0.001" />
    </inertial>
-   <visual>
-    <origin xyz="0 0 0" rpy="0 0 0" />
-    <geometry>
-      <box size="0.001 0.001 0.001" />
-    </geometry>
-   </visual>
-    <collision>
-      <origin xyz="0 0 0" rpy="0 0 0" />
-      <geometry>
-       <box size="0.001 0.001 0.001" />
-      </geometry>
-    </collision>
    </link>
    <joint name="${name}_body_joint" type="fixed">

Commit message: simple base

File: robotino_description/urdf/base.urdf.xacro (robot description, xacro)
@@ -95,5 +95,5 @@
       <origin xyz="0.01 0 0" rpy="0 0 0"/>
       <geometry>
-       <mesh filename="package://robotino_description/meshes/RobotinoBody.stl"/>
+       <cylinder length="0.24" radius="0.23"/>
       </geometry>
     </collision>

Commit message: update

File: robotino_description/urdf/base.urdf.xacro (robot description, xacro)
@@ -93,5 +93,5 @@
     </visual>
     <collision>
-      <origin xyz="0.01 0 0" rpy="0 0 0"/>
+      <origin xyz="0.01 0 0.12" rpy="0 0 0"/>
       <geometry>
        <cylinder length="0.24" radius="0.23"/>

Commit message: set 8 dof

File: robotino_description/urdf/base.urdf.xacro (robot description, xacro)
@@ -6,4 +6,13 @@
   <!--###### IF 8 DOF the joints can be moved ######-->
   <xacro:if value="${has_8dof}">
+  <link name="origin">
+    <inertial>
+      <mass value="10" />
+      <origin xyz="0 0 0" />
+      <inertia ixx="75.0" ixy="0.0" ixz="0.0"
+        iyy="75.0" iyz="0.0"
+        izz="75.0" />
+    </inertial>
+  </link>
    <joint name="origin_joint" type="prismatic">
     <parent link="origin"/>

Commit message: readded 8 dof joints

File: robotino_description/urdf/base.urdf.xacro (robot description, xacro)
@@ -4,7 +4,82 @@
   <xacro:include filename="$(find robotino_description)/urdf/base.transmission.xacro" />
   <xacro:macro name="base" params="name">
-  <link name="${name}_link" />
+  <link name="origin">
+    <inertial>
+      <mass value="10" />
+      <origin xyz="0 0 0" />
+      <inertia ixx="75.0" ixy="0.0" ixz="0.0"
+        iyy="75.0" iyz="0.0"
+        izz="75.0" />
+    </inertial>
+  </link>
+   <joint name="origin_joint" type="prismatic">
+    <parent link="origin"/>
+    <child link="${name}_link"/>
+    <origin xyz="0 0 0" rpy="0 0 0" />
+    <axis xyz="1 0 0" />
+    <limit upper="20" lower="-20" effort="190" velocity="30" />
+   </joint>
+   <link name="${name}_link">
+    <inertial>
+      <mass value="10" />
+      <origin xyz="0 0 0" />
+      <inertia ixx="75.0" ixy="0.0" ixz="0.0"
+       iyy="75.0" iyz="0.0"
+       izz="75.0" />
+    </inertial>
+   </link>
+   <joint name="${name}_jointx" type="prismatic">
+    <parent link="origin"/>
+    <child link="${name}_linkx"/>
+    <origin xyz="0 0 0" rpy="0 0 0" />
+    <axis xyz="1 0 0" />
+    <limit upper="20" lower="-20" effort="0" velocity="0" />
+    <dynamics damping="1000.0" friction="1000.0"/>
+    <safety_controller k_velocity="10" k_position="15" soft_lower_limit="-10.0" soft_upper_limit="10.0" />
+   </joint>
+   <joints_transmission name="base_jointx" />
+   <joint name="${name}_jointy" type="prismatic">
+    <parent link="${name}_linkx"/>
+    <child link="${name}_linky"/>
+    <origin xyz="0 0 0" rpy="0 0 0" />
+    <axis xyz="0 1 0" />
+    <limit upper="20" lower="-20" effort="0" velocity="0" />
+    <dynamics damping="1000.0" friction="1000.0"/>
+    <safety_controller k_velocity="10" k_position="15" soft_lower_limit="-10.0" soft_upper_limit="10.0" />
+   </joint>
+   <joints_transmission name="base_jointy" />
+   <joint name="${name}_jointz" type="revolute">
+    <parent link="${name}_linky"/>
+    <child link="${name}_linkz"/>
+    <origin xyz="0 0 0" rpy="0 0 0" />
+    <axis xyz="0 0 1" />
+    <limit upper="3.14" lower="-3.14" effort="0" velocity="0" />
+    <dynamics damping="1000.0" friction="1000.0"/>
+    <safety_controller k_velocity="10" k_position="15" soft_lower_limit="-3.14" soft_upper_limit="3.14" />
+   </joint>
+   <joints_transmission name="base_jointz" />
+  <link name="${name}_linkx">
+   <inertial>
+    <mass value="0.01"/>
+    <origin xyz="0 0 0"/>
+    <inertia ixx="0.001" ixy="0.0" ixz="0.0" iyy="0.001" iyz="0.0" izz="0.001" />
+   </inertial>
+   </link>
+  <link name="${name}_linky">
+   <inertial>
+    <mass value="0.01"/>
+    <origin xyz="0 0 0"/>
+    <inertia ixx="0.001" ixy="0.0" ixz="0.0" iyy="0.001" iyz="0.0" izz="0.001" />
+   </inertial>
+   </link>
+  <link name="${name}_linkz">
+   <inertial>
+    <mass value="0.01"/>
+    <origin xyz="0 0 0"/>
+    <inertia ixx="0.001" ixy="0.0" ixz="0.0" iyy="0.001" iyz="0.0" izz="0.001" />
+   </inertial>
+   </link>
    <joint name="${name}_body_joint" type="fixed">
-    <parent link="${name}_link"/>
+    <parent link="${name}_linkz"/>
     <child link="${name}_body_link"/>
     <origin xyz="0 0 0" rpy="0 0 0" />
@@ -25,7 +100,7 @@
     </visual>
     <collision>
-      <origin xyz="0.01 0 0" rpy="0 0 0"/>
+      <origin xyz="0.01 0 0.12" rpy="0 0 0"/>
       <geometry>
-       <mesh filename="package://robotino_description/meshes/RobotinoBody.stl"/>
+       <cylinder length="0.24" radius="0.23"/>
       </geometry>
     </collision>
@@ -38,8 +113,8 @@
       <odometryFrame>odom</odometryFrame>
       <odometryRate>20.0</odometryRate>
-      <robotBaseFrame>base_link</robotBaseFrame>
+      <robotBaseFrame>origin</robotBaseFrame>
     </plugin>
   </gazebo>
-   <wheel name="wheel0" parent="base_link">
+   <wheel name="wheel0" parent="base_linkz">
     <origin xyz="0.095 0.14 0.02" rpy="0 0 ${M_PI/3}"/>
     <axis xyz="-1 0 0"/>
@@ -47,5 +122,5 @@
    <wheel_transmission name="wheel0" />
    <wheel_gazebo name="wheel0" />
-   <wheel name="wheel1" parent="base_link">
+   <wheel name="wheel1" parent="base_linkz">
     <origin xyz="-0.16 0 0.02" rpy="0 0 0"/>
     <axis xyz="1 0 0"/>
@@ -53,5 +128,5 @@
    <wheel_transmission name="wheel1" />
    <wheel_gazebo name="wheel1" />
-   <wheel name="wheel2" parent="base_link">
+   <wheel name="wheel2" parent="base_linkz">
     <origin xyz="0.105 -0.15 0.02" rpy="0 0 -${M_PI/3}"/>
     <axis xyz="-1 0 0"/>

Commit message: updates

File: robotino_description/urdf/base.urdf.xacro (robot description, xacro)
@@ -102,5 +102,5 @@
       <origin xyz="0.01 0 0.12" rpy="0 0 0"/>
       <geometry>
-       <cylinder length="0.24" radius="0.23"/>
+	<mesh filename="package://robotino_description/meshes/RobotinoBody.stl"/>
       </geometry>
     </collision>

Commit message: review collisions

File: robotino_description/urdf/base.urdf.xacro (robot description, xacro)
@@ -100,5 +100,5 @@
     </visual>
     <collision>
-      <origin xyz="0.01 0 0.12" rpy="0 0 0"/>
+      <origin xyz="0.01 0 0" rpy="0 0 0"/>
       <geometry>
        <mesh filename="package://robotino_description/meshes/RobotinoBody.stl"/>
