Commit message: update the stl base collision

File: robotino_description/urdf/base.urdf.xacro (robot description, xacro)
@@ -105,4 +105,8 @@
        <mesh filename="package://robotino_description/meshes/RobotinoBody.stl"/>
       </geometry>
+      <!--origin xyz="0.01 0 0.1" rpy="0 0 0"/>
+      <geometry>
+       <cylinder length="0.2" radius="0.2"/>
+      </geometry-->
     </collision>
    </link>
