Commit message: update shell model to be compatible with the calibration software

File: robotino_description/urdf/shell.urdf.xacro (robot description, xacro)
@@ -3,16 +3,14 @@
   <xacro:include filename="$(find robotino_description)/urdf/kinect.urdf.xacro" />
   <xacro:macro name="shell" params="name parent *origin">
-    <joint name="${name}_joint" type="fixed">
+    <joint name="${name}_base_joint" type="fixed">
       <parent link="${parent}"/>
-      <child link="${name}_link" />
+      <child link="${name}_base_link" />
       <insert_block name="origin" />
     </joint>
-   <link name="${name}_link">
+   <link name="${name}_base_link">
       <inertial>
-        <mass value="4" />
-        <origin xyz="0 0 0" />
-        <inertia ixx="75.0" ixy="0.0" ixz="0.0"
-          iyy="75.0" iyz="0.0"
-          izz="75.0" />
+        <mass value="0.01"/>
+        <origin xyz="0 0 0"/>
+        <inertia ixx="0.001" ixy="0.0" ixz="0.0" iyy="0.001" iyz="0.0" izz="0.001" />
       </inertial>
       <visual>
@@ -112,7 +110,4 @@
       </collision>
     </link>
-  <kinect name="kinect" parent="neck_tilt_link">
-    <origin xyz="0 0 0" rpy="-1.57 0 0"/>
-  </kinect>
   </xacro:macro>
 </root>

Commit message: updated the collision model of the shell

File: robotino_description/urdf/shell.urdf.xacro (robot description, xacro)
@@ -24,5 +24,5 @@
       </visual>
       <collision>
-        <origin xyz="0 0 0.05" rpy="0 0 -0.7"/>
+        <origin xyz="0 0 0" rpy="0 0 0"/>
         <geometry>
           <mesh filename="package://robotino_description/meshes/base_shell_collision.stl"/>
@@ -61,5 +61,5 @@
         <origin xyz="0 0 0" rpy="0 0 0"/>
         <geometry>
-          <mesh filename="package://robotino_description/meshes/neck.stl"/>
+          <cylinder length="0.08" radius="0.2"/>
         </geometry>
       </collision>
@@ -104,7 +104,7 @@
       </visual>
       <collision>
-        <origin xyz="0 0 0" rpy="0 0 0"/>
+        <origin xyz="0 0 0.125" rpy="0 0 0"/>
         <geometry>
-          <mesh filename="package://robotino_description/meshes/head.stl"/>
+          <cylinder length="0.25" radius="0.23"/>
         </geometry>
       </collision>

Commit message: add door model

File: robotino_description/urdf/shell.urdf.xacro (robot description, xacro)
@@ -110,4 +110,34 @@
       </collision>
     </link>
+    <joint name="door_joint" type="revolute">
+      <origin xyz="0 0 0" rpy="0 0 0"/>
+      <parent link="${parent}"/>
+      <child link="door_link" />
+      <axis xyz="0 0 1" />
+      <calibration rising="0.1"/>
+      <limit effort="100" lower="0" upper="3.14" velocity="1.4"/>
+    </joint>
+   <link name="door_link">
+      <inertial>
+        <mass value="0.01"/>
+        <origin xyz="0 0 0"/>
+        <inertia ixx="0.001" ixy="0.0" ixz="0.0" iyy="0.001" iyz="0.0" izz="0.001" />
+      </inertial>
+      <visual>
+        <origin xyz="0 0 0" rpy="0 0 0"/>
+        <geometry>
+          <mesh filename="package://robotino_description/meshes/door.stl"/>
+        </geometry>
+        <material name="lightGrey">
+          <color rgba="0.9 0.9 0.9 1"/>
+        </material>
+      </visual>
+      <collision>
+        <origin xyz="0 0 0" rpy="0 0 0"/>
+        <geometry>
+          <mesh filename="package://robotino_description/meshes/door_collision.stl"/>
+        </geometry>
+      </collision>
+    </link>
   </xacro:macro>
 </root>

Commit message: update urdf to support calibration

File: robotino_description/urdf/shell.urdf.xacro (robot description, xacro)
@@ -35,7 +35,13 @@
       <material>Gazebo/LightGrey</material>
     </gazebo>
-    <joint name="neck_pan_joint" type="revolute">
+    <joint name="base_neck_joint" type="fixed">
       <origin xyz="0 0 0.676" rpy="0 0 0"/>
       <parent link="${parent}"/>
+      <child link="base_neck_link" />
+    </joint>
+   <link name="base_neck_link"/>
+    <joint name="neck_pan_joint" type="revolute">
+      <origin xyz="0 0 0" rpy="0 0 0"/>
+      <parent link="base_neck_link"/>
       <child link="neck_pan_link" />
       <axis xyz="0 0 1" />

Commit message: test shell model on real robot

File: robotino_description/urdf/shell.urdf.xacro (robot description, xacro)
@@ -45,5 +45,5 @@
       <parent link="base_neck_link"/>
       <child link="neck_pan_link" />
-      <axis xyz="0 0 1" />
+      <axis xyz="0 0 -1" />
       <calibration rising="0.1"/>
       <limit effort="100" lower="-3.14" upper="3.14" velocity="1.4"/>
@@ -90,5 +90,5 @@
       <parent link="${parent}"/>
       <child link="head_link" />
-      <axis xyz="0 0 1" />
+      <axis xyz="0 0 -1" />
       <calibration rising="0.1"/>
       <limit effort="100" lower="-3.14" upper="3.14" velocity="1.4"/>

Commit message: added gazebo controllers for the shell

File: robotino_description/urdf/shell.urdf.xacro (robot description, xacro)
@@ -30,5 +30,5 @@
       </collision>
     </link>
-    <gazebo reference="${name}_link">
+    <gazebo reference="${name}_base_link">
       <gravity>true</gravity>
       <self_collide>false</self_collide>
@@ -40,5 +40,26 @@
       <child link="base_neck_link" />
     </joint>
-   <link name="base_neck_link"/>
+   <link name="base_neck_link">
+      <inertial>
+        <mass value="0.00001" />
+        <origin xyz="0 0 0" />
+        <inertia ixx="1.0" ixy="0.0" ixz="0.0"
+          iyy="1.0" iyz="0.0"
+          izz="1.0" />
+      </inertial>
+      <visual>
+        <origin xyz="0 0 0" rpy="0 0 0" />
+        <geometry>
+          <box size="0.001 0.001 0.001" />
+        </geometry>
+        <material name="Black"/>
+      </visual>
+      <collision>
+        <origin xyz="0 0 0" rpy="0 0 0" />
+        <geometry>
+          <box size="0.001 0.001 0.001" />
+        </geometry>
+      </collision>
+    </link>
     <joint name="neck_pan_joint" type="revolute">
       <origin xyz="0 0 0" rpy="0 0 0"/>
@@ -146,4 +167,30 @@
       </collision>
     </link>
+    <xacro:shell_transmission name="neck_pan"/>
+    <xacro:shell_transmission name="neck_tilt"/>
+    <xacro:shell_transmission name="head"/>
+    <xacro:shell_transmission name="door"/>
+    <xacro:shell_gazebo name="neck_base"/>
+    <xacro:shell_gazebo name="neck_pan"/>
+    <xacro:shell_gazebo name="neck_tilt"/>
+    <xacro:shell_gazebo name="head"/>
+    <xacro:shell_gazebo name="door"/>
+  </xacro:macro>
+  <xacro:macro name="shell_transmission" params="name">
+    <transmission name="${name}_joint_trans">
+      <type>transmission_interface/SimpleTransmission</type>
+      <joint name="${name}_joint">
+        <hardwareInterface>PositionJointInterface</hardwareInterface>
+      </joint>
+      <actuator name="${name}_joint_motor">
+        <mechanicalReduction>1</mechanicalReduction>
+      </actuator>
+    </transmission>
+  </xacro:macro>
+  <xacro:macro name="shell_gazebo" params="name">
+    <gazebo reference="${name}_link">
+      <gravity>true</gravity>
+      <self_collide>false</self_collide>
+    </gazebo>
   </xacro:macro>
 </root>

Commit message: added a calibration parameter for the neck to the shell

File: robotino_description/urdf/shell.urdf.xacro (robot description, xacro)
@@ -2,5 +2,5 @@
 <root xmlns:xacro="http://www.ros.org/wiki/xacro">
   <xacro:include filename="$(find robotino_description)/urdf/kinect.urdf.xacro" />
-  <xacro:macro name="shell" params="name parent *origin">
+  <xacro:macro name="shell" params="name base_neck_x base_neck_y base_neck_z base_neck_roll base_neck_pitch base_neck_yaw parent *origin">
     <joint name="${name}_base_joint" type="fixed">
       <parent link="${parent}"/>
@@ -36,5 +36,5 @@
     </gazebo>
     <joint name="base_neck_joint" type="fixed">
-      <origin xyz="0 0 0.676" rpy="0 0 0"/>
+      <origin xyz="${base_neck_x} ${base_neck_y} ${base_neck_z}" rpy="${base_neck_roll} ${base_neck_pitch} ${base_neck_yaw}"/>
       <parent link="${parent}"/>
       <child link="base_neck_link" />

Commit message: add front shell collision

File: robotino_description/urdf/shell.urdf.xacro (robot description, xacro)
@@ -27,4 +27,17 @@
         <geometry>
           <mesh filename="package://robotino_description/meshes/base_shell_collision.stl"/>
+        </geometry>
+      </collision>
+    </link>
+    <joint name="${name}_base_joint_front" type="fixed">
+      <parent link="${name}_base_link"/>
+      <child link="${name}_base_link_front" />
+      <origin xyz="0 0 0" rpy="0 0 3.14" />
+    </joint>
+   <link name="${name}_base_link_front">
+      <collision>
+        <origin xyz="0 0 0" rpy="0 0 0"/>
+        <geometry>
+          <mesh filename="package://robotino_description/meshes/base_shell_front_collision.stl"/>
         </geometry>
       </collision>

Commit message: add argument for simulation vs real robot

File: robotino_description/urdf/shell.urdf.xacro (robot description, xacro)
@@ -2,5 +2,5 @@
 <root xmlns:xacro="http://www.ros.org/wiki/xacro">
   <xacro:include filename="$(find robotino_description)/urdf/kinect.urdf.xacro" />
-  <xacro:macro name="shell" params="name base_neck_x base_neck_y base_neck_z base_neck_roll base_neck_pitch base_neck_yaw parent *origin">
+  <xacro:macro name="shell" params="name base_neck_x base_neck_y base_neck_z base_neck_roll base_neck_pitch base_neck_yaw parent *origin real">
     <joint name="${name}_base_joint" type="fixed">
       <parent link="${parent}"/>
@@ -30,4 +30,5 @@
       </collision>
     </link>
+  <xacro:if value="${real}">
     <joint name="${name}_base_joint_front" type="fixed">
       <parent link="${name}_base_link"/>
@@ -43,4 +44,5 @@
       </collision>
     </link>
+  </xacro:if>
     <gazebo reference="${name}_base_link">
       <gravity>true</gravity>

Commit message: use a box as shell front collision

File: robotino_description/urdf/shell.urdf.xacro (robot description, xacro)
@@ -38,7 +38,7 @@
    <link name="${name}_base_link_front">
       <collision>
-        <origin xyz="0 0 0" rpy="0 0 0"/>
-        <geometry>
-          <mesh filename="package://robotino_description/meshes/base_shell_front_collision.stl"/>
+        <origin xyz="-0.02 0 0.085" rpy="0 0 0"/>
+        <geometry>
+          <box size="0.55 0.55 0.17"/>
         </geometry>
       </collision>

Commit message: readded the cylinder collision

File: robotino_description/urdf/shell.urdf.xacro (robot description, xacro)
@@ -38,7 +38,9 @@
    <link name="${name}_base_link_front">
       <collision>
-        <origin xyz="-0.02 0 0.085" rpy="0 0 0"/>
-        <geometry>
-          <box size="0.55 0.55 0.17"/>
+        <!--origin xyz="-0.02 0 0.085" rpy="0 0 0"/-->
+        <origin xyz="0 0 0" rpy="0 0 0"/>
+        <geometry>
+          <mesh filename="package://robotino_description/meshes/base_shell_front_collision.stl"/>
+          <!--box size="0.55 0.55 0.17"/-->
         </geometry>
       </collision>

Commit message: scale shell front collision

File: robotino_description/urdf/shell.urdf.xacro (robot description, xacro)
@@ -41,5 +41,5 @@
         <origin xyz="0 0 0" rpy="0 0 0"/>
         <geometry>
-          <mesh filename="package://robotino_description/meshes/base_shell_front_collision.stl"/>
+          <mesh filename="package://robotino_description/meshes/base_shell_front_collision.stl" scale="1.1 1 1"/>
           <!--box size="0.55 0.55 0.17"/-->
         </geometry>
