Commit message: small fix

File: soft_hand_description/model/soft_hand.urdf.xacro (robot description, xacro)
@@ -402,5 +402,5 @@
       <origin xyz="0 0 0" rpy="0 0 0" />
       <geometry>
-        <mesh filename="package://softhand_description/meshes/wrist.stl" />
+        <mesh filename="package://soft_hand_description/meshes/wrist.stl" />
       </geometry>
       <material name="">
@@ -411,5 +411,5 @@
       <origin xyz="0 0 0" rpy="0 0 0" />
       <geometry>
-        <mesh filename="package://softhand_description/meshes/wrist.stl" />
+        <mesh filename="package://soft_hand_description/meshes/wrist.stl" />
       </geometry>
     </collision>
@@ -426,5 +426,5 @@
       <origin xyz="0 0 0" rpy="0 0 0" />
       <geometry>
-        <mesh filename="package://softhand_description/meshes/robotino_softhand_adapter.stl" />
+        <mesh filename="package://soft_hand_description/meshes/robotino_softhand_adapter.stl" />
       </geometry>
       <material name="">
@@ -435,5 +435,5 @@
       <origin xyz="0 0 0" rpy="0 0 0" />
       <geometry>
-        <mesh filename="package://softhand_description/meshes/robotino_softhand_adapter.stl" />
+        <mesh filename="package://soft_hand_description/meshes/robotino_softhand_adapter.stl" />
       </geometry>
     </collision>

File: soft_hand_description/model/softhand_withCableCanal.urdf.xacro (robot description, xacro)
@@ -25,5 +25,5 @@
       <origin xyz="0 0 0" rpy="0 0 0" />
       <geometry>
-        <mesh filename="package://softhand_description/meshes/cableCanalCollision.stl" />
+        <mesh filename="package://soft_hand_description/meshes/cableCanalCollision.stl" />
       </geometry>
     </collision>

Commit message: missed scala

File: soft_hand_description/model/soft_hand.urdf.xacro (robot description, xacro)
@@ -426,5 +426,5 @@
       <origin xyz="0 0 0" rpy="0 0 0" />
       <geometry>
-        <mesh filename="package://soft_hand_description/meshes/robotino_softhand_adapter.stl" />
+        <mesh filename="package://soft_hand_description/meshes/robotino_softhand_adapter.stl" scale=" .001 .001 .001" />
       </geometry>
       <material name="">
@@ -435,5 +435,5 @@
       <origin xyz="0 0 0" rpy="0 0 0" />
       <geometry>
-        <mesh filename="package://soft_hand_description/meshes/robotino_softhand_adapter.stl" />
+        <mesh filename="package://soft_hand_description/meshes/robotino_softhand_adapter.stl" scale=" .001 .001 .001" />
       </geometry>
     </collision>

Commit message: fixed hand model

File: soft_hand_description/model/soft_hand.urdf.xacro (robot description, xacro)
@@ -400,7 +400,7 @@
       <xacro:default_inertial/>
     <visual>
-      <origin xyz="0 0 0" rpy="0 0 0" />
+      <origin xyz="0 0 0" rpy="1.5708 0 0" />
       <geometry>
-        <mesh filename="package://softhand_description/meshes/wrist.stl" />
+        <mesh filename="package://soft_hand_description/meshes/wrist.stl" />
       </geometry>
       <material name="">
@@ -409,7 +409,7 @@
     </visual>
     <collision>
-      <origin xyz="0 0 0" rpy="0 0 0" />
+      <origin xyz="0 0 0" rpy="1.5708 0 0" />
       <geometry>
-        <mesh filename="package://softhand_description/meshes/wrist.stl" />
+        <mesh filename="package://soft_hand_description/meshes/wrist.stl" />
       </geometry>
     </collision>
@@ -419,12 +419,12 @@
     <parent link="${name}_wrist_link" />
     <child link="${name}_base_link" />
-    </joint>
+  </joint>
   <!-- Angular adapter for SoftHand -->
-  <link name="${name}_base_link">
+  <link parent="${name}_wrist_link" name="${name}_base_link">
       <xacro:default_inertial/>
     <visual>
-      <origin xyz="0 0 0" rpy="0 0 0" />
+      <origin xyz="-0.02 -0.145 0.07" rpy="3.14 0.7854 3.14" />
       <geometry>
-        <mesh filename="package://softhand_description/meshes/robotino_softhand_adapter.stl" />
+        <mesh filename="package://soft_hand_description/meshes/robotino_softhand_adapter_scaled.stl" />
       </geometry>
       <material name="">
@@ -433,7 +433,7 @@
     </visual>
     <collision>
-      <origin xyz="0 0 0" rpy="0 0 0" />
+      <origin xyz="-0.02 -0.145 0.07" rpy="3.14 0.7854 3.14" />
       <geometry>
-        <mesh filename="package://softhand_description/meshes/robotino_softhand_adapter.stl" />
+        <mesh filename="package://soft_hand_description/meshes/robotino_softhand_adapter_scaled.stl" />
       </geometry>
     </collision>
@@ -441,5 +441,5 @@
 		<!-- CLAMP -->
 		<xacro:clamp parent="${name}_base_link" name="${name}_clamp">
-			<origin xyz="0 0 0.01" rpy="0 0 0"/>
+			<origin xyz="-0.02 -0.145 0.07" rpy="0 -0.7854 0"/>
 		</xacro:clamp>
 		<!-- SOFT HAND BASE -->
