Commit message: renamed soft_hand_description package to softhand_description

File: softhand_description/model/accesories/clamp.urdf.xacro (robot description, xacro)
@@ -1,5 +1,5 @@
 <?xml version="1.0"?>
 <robot xmlns:xacro="http://www.ros.org/wiki/xacro">
-<xacro:macro name="softhand_base" params="parent name left *origin">
+<xacro:macro name="clamp" params="parent name *origin">
   <joint name="${parent}_${name}_joint" type="fixed">
     <insert_block name="origin"/>
@@ -11,17 +11,12 @@
       <origin xyz="0 0 0" rpy="0 0 0"/>
       <geometry>
-        <xacro:if value="${left}">
-          <mesh filename="package://soft_hand_description/meshes/accesories/softhand_base_left.stl"/>
-        </xacro:if>
-        <xacro:unless value="${left}">
-          <mesh filename="package://soft_hand_description/meshes/accesories/softhand_base_right.stl"/>
-        </xacro:unless>
+        <mesh filename="package://softhand_description/meshes/accesories/clamp.stl"/>
       </geometry>
       <material name="SoftHand/Blue"/>
     </visual>
     <collision>
-      <origin xyz="0 0 0.031" rpy="0 0 0"/>
+      <origin xyz="0 0 0" rpy="0 0 0"/>
       <geometry>
-        <box size="0.066 0.066 0.062"/>
+        <box size="0.066 0.0725 0.0256"/>
       </geometry>
     </collision>

File: softhand_description/model/accesories/kuka_coupler.urdf.xacro (robot description, xacro)
@@ -11,5 +11,5 @@
       <origin xyz="0 0 0.0115" rpy="0 0 0"/>
       <geometry>
-         <!-- mesh filename="package://soft_hand_description/meshes/accesories/kuka_coupler.stl"/-->
+         <!-- mesh filename="package://softhand_description/meshes/accesories/kuka_coupler.stl"/-->
          <cylinder radius="0.033" length="0.023"/>
       </geometry>

File: softhand_description/model/accesories/softhand_base.urdf.xacro (robot description, xacro)
@@ -1,5 +1,5 @@
 <?xml version="1.0"?>
 <robot xmlns:xacro="http://www.ros.org/wiki/xacro">
-<xacro:macro name="clamp" params="parent name *origin">
+<xacro:macro name="softhand_base" params="parent name left *origin">
   <joint name="${parent}_${name}_joint" type="fixed">
     <insert_block name="origin"/>
@@ -11,12 +11,17 @@
       <origin xyz="0 0 0" rpy="0 0 0"/>
       <geometry>
-        <mesh filename="package://soft_hand_description/meshes/accesories/clamp.stl"/>
+        <xacro:if value="${left}">
+          <mesh filename="package://softhand_description/meshes/accesories/softhand_base_left.stl"/>
+        </xacro:if>
+        <xacro:unless value="${left}">
+          <mesh filename="package://softhand_description/meshes/accesories/softhand_base_right.stl"/>
+        </xacro:unless>
       </geometry>
       <material name="SoftHand/Blue"/>
     </visual>
     <collision>
-      <origin xyz="0 0 0" rpy="0 0 0"/>
+      <origin xyz="0 0 0.031" rpy="0 0 0"/>
       <geometry>
-        <box size="0.066 0.0725 0.0256"/>
+        <box size="0.066 0.066 0.062"/>
       </geometry>
     </collision>

File: softhand_description/model/soft_hand.inertia.xacro (robot description, xacro)
@@ -19,5 +19,5 @@
     </xacro:property>
 <!-- MESHLAB RESULT
-Opened mesh /home/crosales/Code/catkin_ws/src/pisa-iit-soft-hand/soft_hand/soft_hand_description/meshes/knuckle.stl in 9 msec
+Opened mesh /home/crosales/Code/catkin_ws/src/pisa-iit-soft-hand/soft_hand/softhand_description/meshes/knuckle.stl in 9 msec
 All files opened in 1398 msec
 Enabled Decorate mode Show Axis
@@ -46,5 +46,5 @@
     </xacro:property>
 <!-- MESHLAB RESULT
-Opened mesh /home/crosales/Code/catkin_ws/src/pisa-iit-soft-hand/soft_hand/soft_hand_description/meshes/thumb_knuckle.stl in 6 msec
+Opened mesh /home/crosales/Code/catkin_ws/src/pisa-iit-soft-hand/soft_hand/softhand_description/meshes/thumb_knuckle.stl in 6 msec
 All files opened in 1493 msec
 Enabled Decorate mode Show Axis
@@ -73,5 +73,5 @@
     </xacro:property>
 <!-- MESHLAB RESULT
-Opened mesh /home/crosales/Code/catkin_ws/src/pisa-iit-soft-hand/soft_hand/soft_hand_description/meshes/phalanx.stl in 8 msec
+Opened mesh /home/crosales/Code/catkin_ws/src/pisa-iit-soft-hand/soft_hand/softhand_description/meshes/phalanx.stl in 8 msec
 All files opened in 1240 msec
 Mesh Bounding Box Size 25.158094 14.000006 18.515181
@@ -99,5 +99,5 @@
     </xacro:property>
 <!-- MESHLAB RESULT
-Opened mesh /home/crosales/Code/catkin_ws/src/pisa-iit-soft-hand/soft_hand/soft_hand_description/meshes/fingertip.stl in 7 msec
+Opened mesh /home/crosales/Code/catkin_ws/src/pisa-iit-soft-hand/soft_hand/softhand_description/meshes/fingertip.stl in 7 msec
 All files opened in 1241 msec
 Mesh Bounding Box Size 32.299561 14.000006 19.228573
@@ -125,5 +125,5 @@
     </xacro:property>
 <!-- MESHLAB RESULT
-Opened mesh /home/crosales/Code/catkin_ws/src/pisa-iit-soft-hand/soft_hand/soft_hand_description/meshes/palm_right.stl in 13 msec
+Opened mesh /home/crosales/Code/catkin_ws/src/pisa-iit-soft-hand/soft_hand/softhand_description/meshes/palm_right.stl in 13 msec
 All files opened in 1178 msec
 Mesh Bounding Box Size 36.539444 91.129791 84.829025

File: softhand_description/model/soft_hand.urdf.xacro (robot description, xacro)
@@ -2,12 +2,12 @@
 <robot xmlns:xacro="http://ros.org/wiki/xacro">
 	<!-- include other model components -->
-	<xacro:include filename="$(find soft_hand_description)/model/materials.urdf.xacro"/>
-	<xacro:include filename="$(find soft_hand_description)/model/soft_hand.transmission.xacro"/>
-	<xacro:include filename="$(find soft_hand_description)/model/soft_hand.gazebo.xacro"/>
-	<xacro:include filename="$(find soft_hand_description)/model/soft_hand.inertia.xacro"/>
+	<xacro:include filename="$(find softhand_description)/model/materials.urdf.xacro"/>
+	<xacro:include filename="$(find softhand_description)/model/soft_hand.transmission.xacro"/>
+	<xacro:include filename="$(find softhand_description)/model/soft_hand.gazebo.xacro"/>
+	<xacro:include filename="$(find softhand_description)/model/soft_hand.inertia.xacro"/>
 	<!-- accesories -->
-	<xacro:include filename="$(find soft_hand_description)/model/accesories/kuka_coupler.urdf.xacro"/>
-	<xacro:include filename="$(find soft_hand_description)/model/accesories/clamp.urdf.xacro"/>
-	<xacro:include filename="$(find soft_hand_description)/model/accesories/softhand_base.urdf.xacro"/>
+	<xacro:include filename="$(find softhand_description)/model/accesories/kuka_coupler.urdf.xacro"/>
+	<xacro:include filename="$(find softhand_description)/model/accesories/clamp.urdf.xacro"/>
+	<xacro:include filename="$(find softhand_description)/model/accesories/softhand_base.urdf.xacro"/>
 	<xacro:property name="pi" value="3.1415926535897931" />
 	<!-- joint properties -->
@@ -80,5 +80,5 @@
 			<visual>
 				<geometry>
-					<mesh filename="package://soft_hand_description/meshes/knuckle.stl" scale=" .001 .001 .001" />
+					<mesh filename="package://softhand_description/meshes/knuckle.stl" scale=" .001 .001 .001" />
 				</geometry>
 				<material name="SoftHand/DarkGrey" />
@@ -86,5 +86,5 @@
 			<collision>
 				<geometry>
-					<mesh filename="package://soft_hand_description/meshes/knuckle_collision.stl" scale=" .001 .001 .001" />
+					<mesh filename="package://softhand_description/meshes/knuckle_collision.stl" scale=" .001 .001 .001" />
 				</geometry>
 			</collision>
@@ -124,5 +124,5 @@
 			<visual>
 				<geometry>
-					<mesh filename="package://soft_hand_description/meshes/phalanx.stl" scale=" .001 .001 .001" />
+					<mesh filename="package://softhand_description/meshes/phalanx.stl" scale=" .001 .001 .001" />
 				</geometry>
 				<material name="SoftHand/DarkGrey" />
@@ -130,5 +130,5 @@
 			<collision>
 				<geometry>
-					<mesh filename="package://soft_hand_description/meshes/phalanx_collision.stl" scale=" .001 .001 .001" />
+					<mesh filename="package://softhand_description/meshes/phalanx_collision.stl" scale=" .001 .001 .001" />
 				</geometry>
 			</collision>
@@ -168,5 +168,5 @@
 			<visual>
 				<geometry>
-					<mesh filename="package://soft_hand_description/meshes/phalanx.stl" scale=" .001 .001 .001" />
+					<mesh filename="package://softhand_description/meshes/phalanx.stl" scale=" .001 .001 .001" />
 				</geometry>
 				<material name="SoftHand/DarkGrey" />
@@ -174,5 +174,5 @@
 			<collision>
 				<geometry>
-					<mesh filename="package://soft_hand_description/meshes/phalanx_collision.stl" scale=" .001 .001 .001" />
+					<mesh filename="package://softhand_description/meshes/phalanx_collision.stl" scale=" .001 .001 .001" />
 				</geometry>
 			</collision>
@@ -212,5 +212,5 @@
 			<visual>
 				<geometry>
-					<mesh filename="package://soft_hand_description/meshes/fingertip.stl" scale=" .001 .001 .001" />
+					<mesh filename="package://softhand_description/meshes/fingertip.stl" scale=" .001 .001 .001" />
 				</geometry>
 				<material name="SoftHand/DarkGrey" />
@@ -218,5 +218,5 @@
 			<collision>
 				<geometry>
-					<mesh filename="package://soft_hand_description/meshes/fingertip_collision.stl" scale=" .001 .001 .001" />
+					<mesh filename="package://softhand_description/meshes/fingertip_collision.stl" scale=" .001 .001 .001" />
 				</geometry>
 			</collision>
@@ -245,5 +245,5 @@
 				<visual>
 					<geometry>
-						<mesh filename="package://soft_hand_description/meshes/thumb_knuckle_left.stl" scale=" .001 .001 .001" />
+						<mesh filename="package://softhand_description/meshes/thumb_knuckle_left.stl" scale=" .001 .001 .001" />
 					</geometry>
 					<material name="SoftHand/DarkGrey" />
@@ -251,5 +251,5 @@
 				<collision>
 					<geometry>
-						<mesh filename="package://soft_hand_description/meshes/thumb_knuckle_left_collision.stl" scale=" .001 .001 .001" />
+						<mesh filename="package://softhand_description/meshes/thumb_knuckle_left_collision.stl" scale=" .001 .001 .001" />
 					</geometry>
 				</collision>
@@ -287,5 +287,5 @@
 				<visual>
 					<geometry>
-						<mesh filename="package://soft_hand_description/meshes/thumb_knuckle_right.stl" scale=" .001 .001 .001" />
+						<mesh filename="package://softhand_description/meshes/thumb_knuckle_right.stl" scale=" .001 .001 .001" />
 					</geometry>
 					<material name="SoftHand/DarkGrey" />
@@ -293,5 +293,5 @@
 				<collision>
 					<geometry>
-						<mesh filename="package://soft_hand_description/meshes/thumb_knuckle_right_collision.stl" scale=" .001 .001 .001" />
+						<mesh filename="package://softhand_description/meshes/thumb_knuckle_right_collision.stl" scale=" .001 .001 .001" />
 					</geometry>
 				</collision>
@@ -333,5 +333,5 @@
 			<visual>
 				<geometry>
-					<mesh filename="package://soft_hand_description/meshes/phalanx.stl" scale=" .001 .001 .001" />
+					<mesh filename="package://softhand_description/meshes/phalanx.stl" scale=" .001 .001 .001" />
 				</geometry>
 				<material name="SoftHand/DarkGrey" />
@@ -339,5 +339,5 @@
 			<collision>
 				<geometry>
-					<mesh filename="package://soft_hand_description/meshes/phalanx_collision.stl" scale=" .001 .001 .001" />
+					<mesh filename="package://softhand_description/meshes/phalanx_collision.stl" scale=" .001 .001 .001" />
 				</geometry>
 			</collision>
@@ -377,5 +377,5 @@
 			<visual>
 				<geometry>
-					<mesh filename="package://soft_hand_description/meshes/fingertip.stl" scale=" .001 .001 .001" />
+					<mesh filename="package://softhand_description/meshes/fingertip.stl" scale=" .001 .001 .001" />
 				</geometry>
 				<material name="SoftHand/DarkGrey" />
@@ -383,5 +383,5 @@
 			<collision>
 				<geometry>
-					<mesh filename="package://soft_hand_description/meshes/fingertip_collision.stl" scale=" .001 .001 .001" />
+					<mesh filename="package://softhand_description/meshes/fingertip_collision.stl" scale=" .001 .001 .001" />
 				</geometry>
 			</collision>
@@ -402,5 +402,5 @@
       <origin xyz="0 0 0" rpy="1.5708 0 0" />
       <geometry>
-        <mesh filename="package://soft_hand_description/meshes/wrist.stl" />
+        <mesh filename="package://softhand_description/meshes/wrist.stl" />
       </geometry>
       <material name="">
@@ -411,5 +411,5 @@
       <origin xyz="0 0 0" rpy="1.5708 0 0" />
       <geometry>
-        <mesh filename="package://soft_hand_description/meshes/wrist.stl" />
+        <mesh filename="package://softhand_description/meshes/wrist.stl" />
       </geometry>
     </collision>
@@ -426,5 +426,5 @@
       <origin xyz="-0.02 -0.145 0.07" rpy="3.14 0.7854 3.14" />
       <geometry>
-        <mesh filename="package://soft_hand_description/meshes/robotino_softhand_adapter_scaled.stl" />
+        <mesh filename="package://softhand_description/meshes/robotino_softhand_adapter_scaled.stl" />
       </geometry>
       <material name="">
@@ -435,5 +435,5 @@
       <origin xyz="-0.02 -0.145 0.07" rpy="3.14 0.7854 3.14" />
       <geometry>
-        <mesh filename="package://soft_hand_description/meshes/robotino_softhand_adapter_scaled.stl" />
+        <mesh filename="package://softhand_description/meshes/robotino_softhand_adapter_scaled.stl" />
       </geometry>
     </collision>
@@ -465,5 +465,5 @@
 				<visual>
 					<geometry>
-						<mesh filename="package://soft_hand_description/meshes/palm_left.stl" scale=" .001 .001 .001" />
+						<mesh filename="package://softhand_description/meshes/palm_left.stl" scale=" .001 .001 .001" />
 					</geometry>
 					<material name="SoftHand/DarkGrey" />
@@ -471,5 +471,5 @@
 				<collision>
 					<geometry>
-						<mesh filename="package://soft_hand_description/meshes/palm_left_collision.stl" scale=" .001 .001 .001" />
+						<mesh filename="package://softhand_description/meshes/palm_left_collision.stl" scale=" .001 .001 .001" />
 					</geometry>
 				</collision>
@@ -478,5 +478,5 @@
 				<visual>
 					<geometry>
-						<mesh filename="package://soft_hand_description/meshes/palm_right.stl" scale=" .001 .001 .001" />
+						<mesh filename="package://softhand_description/meshes/palm_right.stl" scale=" .001 .001 .001" />
 					</geometry>
 					<material name="SoftHand/DarkGrey" />
@@ -484,5 +484,5 @@
 				<collision>
 					<geometry>
-						<mesh filename="package://soft_hand_description/meshes/palm_right_collision.stl" scale=" .001 .001 .001" />
+						<mesh filename="package://softhand_description/meshes/palm_right_collision.stl" scale=" .001 .001 .001" />
 					</geometry>
 				</collision>
