Commit message: renamed soft_hand_description package to softhand_description

File: softhand_description/model/soft_hand_fixed.urdf.xacro (robot description, xacro)
@@ -2,12 +2,12 @@
 <robot xmlns:xacro="http://ros.org/wiki/xacro">
 	<!-- include other model components -->
-	<xacro:include filename="$(find soft_hand_description)/model/materials.urdf.xacro"/>
-	<xacro:include filename="$(find soft_hand_description)/model/soft_hand.transmission.xacro"/>
-	<xacro:include filename="$(find soft_hand_description)/model/soft_hand.gazebo.xacro"/>
-	<xacro:include filename="$(find soft_hand_description)/model/soft_hand.inertia.xacro"/>
+	<xacro:include filename="$(find softhand_description)/model/materials.urdf.xacro"/>
+	<xacro:include filename="$(find softhand_description)/model/soft_hand.transmission.xacro"/>
+	<xacro:include filename="$(find softhand_description)/model/soft_hand.gazebo.xacro"/>
+	<xacro:include filename="$(find softhand_description)/model/soft_hand.inertia.xacro"/>
 	<!-- accesories -->
-	<xacro:include filename="$(find soft_hand_description)/model/accesories/kuka_coupler.urdf.xacro"/>
-	<xacro:include filename="$(find soft_hand_description)/model/accesories/clamp.urdf.xacro"/>
-	<xacro:include filename="$(find soft_hand_description)/model/accesories/softhand_base.urdf.xacro"/>
+	<xacro:include filename="$(find softhand_description)/model/accesories/kuka_coupler.urdf.xacro"/>
+	<xacro:include filename="$(find softhand_description)/model/accesories/clamp.urdf.xacro"/>
+	<xacro:include filename="$(find softhand_description)/model/accesories/softhand_base.urdf.xacro"/>
 	<xacro:property name="pi" value="3.1415926535897931" />
 	<!-- joint properties -->
@@ -81,5 +81,5 @@
 			<visual>
 				<geometry>
-					<mesh filename="package://soft_hand_description/meshes/knuckle.stl" scale=" .001 .001 .001" />
+					<mesh filename="package://softhand_description/meshes/knuckle.stl" scale=" .001 .001 .001" />
 				</geometry>
 				<material name="SoftHand/DarkGrey" />
@@ -87,5 +87,5 @@
 			<collision>
 				<geometry>
-					<mesh filename="package://soft_hand_description/meshes/knuckle_collision.stl" scale=" .001 .001 .001" />
+					<mesh filename="package://softhand_description/meshes/knuckle_collision.stl" scale=" .001 .001 .001" />
 				</geometry>
 			</collision>
@@ -125,5 +125,5 @@
 			<visual>
 				<geometry>
-					<mesh filename="package://soft_hand_description/meshes/phalanx.stl" scale=" .001 .001 .001" />
+					<mesh filename="package://softhand_description/meshes/phalanx.stl" scale=" .001 .001 .001" />
 				</geometry>
 				<material name="SoftHand/DarkGrey" />
@@ -131,5 +131,5 @@
 			<collision>
 				<geometry>
-					<mesh filename="package://soft_hand_description/meshes/phalanx_collision.stl" scale=" .001 .001 .001" />
+					<mesh filename="package://softhand_description/meshes/phalanx_collision.stl" scale=" .001 .001 .001" />
 				</geometry>
 			</collision>
@@ -169,5 +169,5 @@
 			<visual>
 				<geometry>
-					<mesh filename="package://soft_hand_description/meshes/phalanx.stl" scale=" .001 .001 .001" />
+					<mesh filename="package://softhand_description/meshes/phalanx.stl" scale=" .001 .001 .001" />
 				</geometry>
 				<material name="SoftHand/DarkGrey" />
@@ -175,5 +175,5 @@
 			<collision>
 				<geometry>
-					<mesh filename="package://soft_hand_description/meshes/phalanx_collision.stl" scale=" .001 .001 .001" />
+					<mesh filename="package://softhand_description/meshes/phalanx_collision.stl" scale=" .001 .001 .001" />
 				</geometry>
 			</collision>
@@ -213,5 +213,5 @@
 			<visual>
 				<geometry>
-					<mesh filename="package://soft_hand_description/meshes/fingertip.stl" scale=" .001 .001 .001" />
+					<mesh filename="package://softhand_description/meshes/fingertip.stl" scale=" .001 .001 .001" />
 				</geometry>
 				<material name="SoftHand/DarkGrey" />
@@ -219,5 +219,5 @@
 			<collision>
 				<geometry>
-					<mesh filename="package://soft_hand_description/meshes/fingertip_collision.stl" scale=" .001 .001 .001" />
+					<mesh filename="package://softhand_description/meshes/fingertip_collision.stl" scale=" .001 .001 .001" />
 				</geometry>
 			</collision>
@@ -246,5 +246,5 @@
 				<visual>
 					<geometry>
-						<mesh filename="package://soft_hand_description/meshes/thumb_knuckle_left.stl" scale=" .001 .001 .001" />
+						<mesh filename="package://softhand_description/meshes/thumb_knuckle_left.stl" scale=" .001 .001 .001" />
 					</geometry>
 					<material name="SoftHand/DarkGrey" />
@@ -252,5 +252,5 @@
 				<collision>
 					<geometry>
-						<mesh filename="package://soft_hand_description/meshes/thumb_knuckle_left_collision.stl" scale=" .001 .001 .001" />
+						<mesh filename="package://softhand_description/meshes/thumb_knuckle_left_collision.stl" scale=" .001 .001 .001" />
 					</geometry>
 				</collision>
@@ -288,5 +288,5 @@
 				<visual>
 					<geometry>
-						<mesh filename="package://soft_hand_description/meshes/thumb_knuckle_right.stl" scale=" .001 .001 .001" />
+						<mesh filename="package://softhand_description/meshes/thumb_knuckle_right.stl" scale=" .001 .001 .001" />
 					</geometry>
 					<material name="SoftHand/DarkGrey" />
@@ -294,5 +294,5 @@
 				<collision>
 					<geometry>
-						<mesh filename="package://soft_hand_description/meshes/thumb_knuckle_right_collision.stl" scale=" .001 .001 .001" />
+						<mesh filename="package://softhand_description/meshes/thumb_knuckle_right_collision.stl" scale=" .001 .001 .001" />
 					</geometry>
 				</collision>
@@ -334,5 +334,5 @@
 			<visual>
 				<geometry>
-					<mesh filename="package://soft_hand_description/meshes/phalanx.stl" scale=" .001 .001 .001" />
+					<mesh filename="package://softhand_description/meshes/phalanx.stl" scale=" .001 .001 .001" />
 				</geometry>
 				<material name="SoftHand/DarkGrey" />
@@ -340,5 +340,5 @@
 			<collision>
 				<geometry>
-					<mesh filename="package://soft_hand_description/meshes/phalanx_collision.stl" scale=" .001 .001 .001" />
+					<mesh filename="package://softhand_description/meshes/phalanx_collision.stl" scale=" .001 .001 .001" />
 				</geometry>
 			</collision>
@@ -378,5 +378,5 @@
 			<visual>
 				<geometry>
-					<mesh filename="package://soft_hand_description/meshes/fingertip.stl" scale=" .001 .001 .001" />
+					<mesh filename="package://softhand_description/meshes/fingertip.stl" scale=" .001 .001 .001" />
 				</geometry>
 				<material name="SoftHand/DarkGrey" />
@@ -384,5 +384,5 @@
 			<collision>
 				<geometry>
-					<mesh filename="package://soft_hand_description/meshes/fingertip_collision.stl" scale=" .001 .001 .001" />
+					<mesh filename="package://softhand_description/meshes/fingertip_collision.stl" scale=" .001 .001 .001" />
 				</geometry>
 			</collision>
@@ -403,5 +403,5 @@
       <origin xyz="0 0 0" rpy="1.5708 0 0" />
       <geometry>
-        <mesh filename="package://soft_hand_description/meshes/wrist.stl" />
+        <mesh filename="package://softhand_description/meshes/wrist.stl" />
       </geometry>
       <material name="">
@@ -412,5 +412,5 @@
       <origin xyz="0 0 0" rpy="1.5708 0 0" />
       <geometry>
-        <mesh filename="package://soft_hand_description/meshes/wrist.stl" />
+        <mesh filename="package://softhand_description/meshes/wrist.stl" />
       </geometry>
     </collision>
@@ -427,5 +427,5 @@
       <origin xyz="-0.02 -0.145 0.07" rpy="3.14 0.7854 3.14" />
       <geometry>
-        <mesh filename="package://soft_hand_description/meshes/robotino_softhand_adapter_scaled.stl" />
+        <mesh filename="package://softhand_description/meshes/robotino_softhand_adapter_scaled.stl" />
       </geometry>
       <material name="">
@@ -436,5 +436,5 @@
       <origin xyz="-0.02 -0.145 0.07" rpy="3.14 0.7854 3.14" />
       <geometry>
-        <mesh filename="package://soft_hand_description/meshes/robotino_softhand_adapter_scaled.stl" />
+        <mesh filename="package://softhand_description/meshes/robotino_softhand_adapter_scaled.stl" />
       </geometry>
     </collision>
@@ -466,5 +466,5 @@
 				<visual>
 					<geometry>
-						<mesh filename="package://soft_hand_description/meshes/palm_left.stl" scale=" .001 .001 .001" />
+						<mesh filename="package://softhand_description/meshes/palm_left.stl" scale=" .001 .001 .001" />
 					</geometry>
 					<material name="SoftHand/DarkGrey" />
@@ -472,5 +472,5 @@
 				<collision>
 					<geometry>
-						<mesh filename="package://soft_hand_description/meshes/palm_left_collision.stl" scale=" .001 .001 .001" />
+						<mesh filename="package://softhand_description/meshes/palm_left_collision.stl" scale=" .001 .001 .001" />
 					</geometry>
 				</collision>
@@ -479,5 +479,5 @@
 				<visual>
 					<geometry>
-						<mesh filename="package://soft_hand_description/meshes/palm_right.stl" scale=" .001 .001 .001" />
+						<mesh filename="package://softhand_description/meshes/palm_right.stl" scale=" .001 .001 .001" />
 					</geometry>
 					<material name="SoftHand/DarkGrey" />
@@ -485,5 +485,5 @@
 				<collision>
 					<geometry>
-						<mesh filename="package://soft_hand_description/meshes/palm_right_collision.stl" scale=" .001 .001 .001" />
+						<mesh filename="package://softhand_description/meshes/palm_right_collision.stl" scale=" .001 .001 .001" />
 					</geometry>
 				</collision>

File: softhand_description/model/softhand_withCableCanal.urdf.xacro (robot description, xacro)
@@ -1,5 +1,5 @@
 <?xml version="1.0"?>
 <robot xmlns:xacro="http://www.ros.org/wiki/xacro">
-  <xacro:include filename="$(find soft_hand_description)/model/soft_hand_fixed.urdf.xacro" />
+  <xacro:include filename="$(find softhand_description)/model/soft_hand_fixed.urdf.xacro" />
   <xacro:macro name="softhand" params="parent name withAdaptiveTransmission useMimicTag left *origin">
   <xacro:soft_hand name="${name}" parent="softhand_base_link" withAdaptiveTransmission="false" useMimicTag="false" left="false">
@@ -25,5 +25,5 @@
       <origin xyz="0 0 0" rpy="0 0 0" />
       <geometry>
-        <mesh filename="package://soft_hand_description/meshes/cableCanalCollision.stl" />
+        <mesh filename="package://softhand_description/meshes/cableCanalCollision.stl" />
       </geometry>
     </collision>
